File: Hardware/synth_psoc.kicad_pcb (KiCad board)
At the start: 2 copper layers, 1 part, among them Q1 Q_PJFET_DGS

Commit message: measure positions of potentiometers and tentative board edge definition.
Parts:
- added C1: 1uF, Capacitors_SMD:CP_Elec_4x4.5, F.Cu at (412.6, 138.7)
- added C10: 22uF, Capacitors_SMD:CP_Elec_5x5.7, F.Cu at (404.9, 151.3)
- added C11: 22uF, Capacitors_SMD:CP_Elec_5x5.7, F.Cu at (408.0, 119.4)
- added C12: 22uF, Capacitors_SMD:CP_Elec_5x5.7, F.Cu at (421.3, 109.5)
- added C13: 22uF, Capacitors_SMD:CP_Elec_5x5.7, F.Cu at (399.6, 131.6)
- added C14: 22uF, Capacitors_SMD:CP_Elec_5x5.7, F.Cu at (379.8, 148.9)
- added C15: 22uF, Capacitors_SMD:CP_Elec_5x5.7, F.Cu at (388.2, 139.0)
- added C16: 100p, digikey-footprints:0805, F.Cu at (422.6, 137.1)
- added C17: 100p, digikey-footprints:0805, F.Cu at (418.3, 143.0)
- added C18: 100p, digikey-footprints:0805, F.Cu at (429.8, 127.2)
- added C19: 22uF, Capacitors_SMD:CP_Elec_5x5.7, F.Cu at (379.8, 139.0)
- added C2: 1uF, Capacitors_SMD:CP_Elec_4x4.5, F.Cu at (432.4, 119.0)
- added C20: 22uF, Capacitors_SMD:CP_Elec_5x5.7, F.Cu at (404.6, 109.5)
- added C21: 22uF, Capacitors_SMD:CP_Elec_5x5.7, F.Cu at (412.9, 109.5)
- added C22: 1uF, Capacitors_SMD:CP_Elec_4x4.5, F.Cu at (424.1, 128.8)
- added C23: 22uF, Capacitors_SMD:CP_Elec_5x5.7, F.Cu at (396.5, 141.4)
- added C24: 22uF, Capacitors_SMD:CP_Elec_5x5.7, F.Cu at (429.6, 109.5)
- added C25: 22uF, Capacitors_SMD:CP_Elec_5x5.7, F.Cu at (404.9, 141.4)
- added C26: 22uF, Capacitors_SMD:CP_Elec_5x5.7, F.Cu at (416.3, 129.3)
- added C27: 100p, digikey-footprints:0805, F.Cu at (418.3, 137.1)
- added C28: 22uF, Capacitors_SMD:CP_Elec_5x5.7, F.Cu at (424.7, 119.4)
- added C29: 220uF, Capacitors_SMD:CP_Elec_8x10, F.Cu at (490.5, -31.4)
- added C3: 1uF, Capacitors_SMD:CP_Elec_4x4.5, F.Cu at (445.7, 109.1)
- added C30: 1uF, Capacitors_SMD:CP_Elec_4x4.5, F.Cu at (493.2, -19.6)
- added C31: 4.7uF, Capacitors_SMD:CP_Elec_4x5.7, F.Cu at (500.6, -18.5)
- added C32: 220u, Capacitors_SMD:CP_Elec_8x10, F.Cu at (488.4, 85.9)
- added C33: 220u, Capacitors_SMD:CP_Elec_8x10, F.Cu at (499.5, 73.0)
- added C34: 220u, Capacitors_SMD:CP_Elec_8x10, F.Cu at (518.1, 55.6)
- added C35: 220u, Capacitors_SMD:CP_Elec_8x10, F.Cu at (462.5, 90.3)
- added C36: 220u, Capacitors_SMD:CP_Elec_8x10, F.Cu at (477.4, 73.0)
- added C37: 220u, Capacitors_SMD:CP_Elec_8x10, F.Cu at (488.4, 73.0)
- added C38: 220u, Capacitors_SMD:CP_Elec_8x10, F.Cu at (477.4, 85.9)
- added C39: 220u, Capacitors_SMD:CP_Elec_8x10, F.Cu at (507.1, 55.6)
- added C4: 22uF, Capacitors_SMD:CP_Elec_5x5.7, F.Cu at (408.0, 129.3)
- added C40: 1nF, digikey-footprints:0805, F.Cu at (547.0, 69.5)
- added C41: 1nF, digikey-footprints:0805, F.Cu at (521.4, 95.2)
- added C42: 1nF, digikey-footprints:0805, F.Cu at (525.8, 89.3)
- added C43: 1nF, digikey-footprints:0805, F.Cu at (538.1, 75.4)
- added C44: 22uF, Capacitors_SMD:CP_Elec_5x5.7, F.Cu at (498.1, 94.3)
- added C45: 22uF, Capacitors_SMD:CP_Elec_5x5.7, F.Cu at (519.1, 67.0)
- added C46: 22uF, Capacitors_SMD:CP_Elec_5x5.7, F.Cu at (498.1, 84.4)
- added C47: 22uF, Capacitors_SMD:CP_Elec_5x5.7, F.Cu at (527.8, 54.1)
- added C48: 22uF, Capacitors_SMD:CP_Elec_5x5.7, F.Cu at (509.2, 79.2)
- added C49: 22uF, Capacitors_SMD:CP_Elec_5x5.7, F.Cu at (536.2, 54.1)
- added C5: 22uF, Capacitors_SMD:CP_Elec_5x5.7, F.Cu at (416.3, 119.4)
- added C50: 22uF, Capacitors_SMD:CP_Elec_5x5.7, F.Cu at (527.8, 64.0)
- added C51: 22uF, Capacitors_SMD:CP_Elec_5x5.7, F.Cu at (506.5, 89.1)
- added C52: 22uF, Capacitors_SMD:CP_Elec_5x5.7, F.Cu at (398.5, 164.8)
- added C53: 22uF, Capacitors_SMD:CP_Elec_5x5.7, F.Cu at (390.1, 164.8)
- added C54: 22uF, Capacitors_SMD:CP_Elec_5x5.7, F.Cu at (381.4, 174.7)
- added C55: 22uF, Capacitors_SMD:CP_Elec_5x5.7, F.Cu at (373.0, 174.5)
- added C56: 100pF, digikey-footprints:0805, F.Cu at (392.3, 178.5)
- added C57: 22uF, Capacitors_SMD:CP_Elec_5x5.7, F.Cu at (381.8, 164.8)
- added C58: 22uF, Capacitors_SMD:CP_Elec_5x5.7, F.Cu at (538.3, 119.4)
- added C59: 220uF, Capacitors_SMD:CP_Elec_8x10, F.Cu at (477.1, 145.8)
- added C6: 22uF, Capacitors_SMD:CP_Elec_5x5.7, F.Cu at (396.5, 151.3)
- added C60: 22uF, Capacitors_SMD:CP_Elec_5x5.7, F.Cu at (509.8, 144.2)
- added C61: 22uF, Capacitors_SMD:CP_Elec_5x5.7, F.Cu at (538.3, 109.5)
- added C62: 33nF, digikey-footprints:0805, F.Cu at (467.4, 151.1)
- added C63: 33nF, digikey-footprints:0805, F.Cu at (463.1, 151.1)
- added C64: 22uF, Capacitors_SMD:CP_Elec_5x5.7, F.Cu at (520.3, 126.9)
- added C65: 220uF, Capacitors_SMD:CP_Elec_8x10, F.Cu at (488.2, 145.8)
- added C66: 22uF, Capacitors_SMD:CP_Elec_5x5.7, F.Cu at (528.7, 126.9)
- added C67: 22uF, Capacitors_SMD:CP_Elec_5x5.7, F.Cu at (520.3, 136.8)
- added C68: 33nF, digikey-footprints:0805, F.Cu at (530.8, 145.8)
- added C69: 33nF, digikey-footprints:0805, F.Cu at (500.1, 152.0)
- added C7: 22uF, Capacitors_SMD:CP_Elec_5x5.7, F.Cu at (399.6, 121.7)
- added C70: 22uF, Capacitors_SMD:CP_Elec_5x5.7, F.Cu at (537.0, 129.3)
- added C71: 22uF, Capacitors_SMD:CP_Elec_5x5.7, F.Cu at (528.7, 136.8)
- added C72: 22pF, digikey-footprints:0805, F.Cu at (114.2, 174.4)
- added C73: 22pF, digikey-footprints:0805, F.Cu at (114.2, 149.0)
- added C8: 22uF, Capacitors_SMD:CP_Elec_5x5.7, F.Cu at (438.0, 109.5)
- added C9: 22uF, Capacitors_SMD:CP_Elec_5x5.7, F.Cu at (388.2, 148.9)
- added D1: D, digikey-footprints:TO-252-3, F.Cu at (466.2, -44.3)
- added D2: BZX84C3V3-T1, digikey-footprints:SOT-23-3, F.Cu at (499.6, 143.7)
- added J1: Barrel_Jack, Connectors:BARREL_JACK, F.Cu at (453.9, -37.5)
- added J2: Audio-Jack-2_Switch, Connectors:PINHEAD1-3, F.Cu at (366.7, 164.7)
- added J3: SWD_programming, Pin_Headers:Pin_Header_Straight_1x05_Pitch2.54mm, F.Cu at (104.1, 170.2)
- added Q2: MMBFJ177, digikey-footprints:SOT-23-3, F.Cu at (488.4, 96.8)
- added Q3: MMBFJ177, digikey-footprints:SOT-23-3, F.Cu at (480.3, 96.8)
- added Q4: MMBFJ177, digikey-footprints:SOT-23-3, F.Cu at (472.1, 96.8)
- added Q5: 2N3904, digikey-footprints:SOT-23-3, F.Cu at (517.0, 146.1)
- added Q6: 2N3904, digikey-footprints:SOT-23-3, F.Cu at (545.5, 118.8)
- added Q7: 2N3904, digikey-footprints:SOT-23-3, F.Cu at (535.9, 138.7)
- added Q8: 2N3904, digikey-footprints:SOT-23-3, F.Cu at (545.5, 127.5)
- added R1: 1k, digikey-footprints:0805, F.Cu at (451.0, 119.1)
- added R10: 10k, digikey-footprints:0805, F.Cu at (411.2, 152.0)
- added R100: R, digikey-footprints:0805, F.Cu at (447.4, 57.9)
- added R101: R, digikey-footprints:0805, F.Cu at (443.2, 63.7)
- added R102: R, digikey-footprints:0805, F.Cu at (437.5, 69.4)
- added R103: R, digikey-footprints:0805, F.Cu at (447.4, 63.7)
- added R104: R, digikey-footprints:0805, F.Cu at (451.7, 57.9)
- added R105: R, digikey-footprints:0805, F.Cu at (451.7, 63.7)
- added R11: 10k, digikey-footprints:0805, F.Cu at (429.8, 133.1)
- added R12: 10k, digikey-footprints:0805, F.Cu at (438.3, 123.2)
- added R13: 10k, digikey-footprints:0805, F.Cu at (451.4, 113.3)
- added R14: 10k, digikey-footprints:0805, F.Cu at (422.6, 143.0)
- added R15: 10k, digikey-footprints:0805, F.Cu at (451.4, 107.5)
- added R16: 470k, digikey-footprints:0805, F.Cu at (435.3, 143.9)
- added R17: 470k, digikey-footprints:0805, F.Cu at (446.6, 116.5)
- added R18: 470k, digikey-footprints:0805, F.Cu at (431.1, 144.8)
- added R19: 10k, digikey-footprints:0805, F.Cu at (434.0, 126.4)
- added R2: 1k, digikey-footprints:0805, F.Cu at (431.1, 138.9)
- added R20: 10k, digikey-footprints:0805, F.Cu at (426.8, 138.9)
- added R21: 10k, digikey-footprints:0805, F.Cu at (439.6, 140.7)
- added R22: 100k, digikey-footprints:0805, F.Cu at (428.2, 150.6)
- added R23: 100k, digikey-footprints:0805, F.Cu at (442.4, 117.3)
- added R24: 100k, digikey-footprints:0805, F.Cu at (443.8, 134.9)
- added R25: 1k, digikey-footprints:0805, F.Cu at (411.2, 146.2)
- added R26: 470k, digikey-footprints:0805, F.Cu at (439.6, 134.9)
- added R27: 470k, digikey-footprints:0805, F.Cu at (423.9, 150.6)
- added R28: 10k, digikey-footprints:0805, F.Cu at (451.0, 125.0)
- added R29: 10k, digikey-footprints:0805, F.Cu at (426.8, 144.8)
- added R3: 1k, digikey-footprints:0805, F.Cu at (438.1, 117.3)
- added R30: 470k, digikey-footprints:0805, F.Cu at (442.5, 129.0)
- added R31: 10k, digikey-footprints:0805, F.Cu at (446.8, 128.2)
- added R32: 100k, digikey-footprints:0805, F.Cu at (435.3, 138.1)
- added R33: 100k, digikey-footprints:0805, F.Cu at (474.5, -28.9)
- added R34: 100k, digikey-footprints:0805, F.Cu at (481.3, -32.0)
- added R35: 22k, digikey-footprints:0805, F.Cu at (529.6, 71.8)
- added R36: 22k, digikey-footprints:0805, F.Cu at (512.8, 93.6)
- added R37: 470k, digikey-footprints:0805, F.Cu at (517.0, 87.7)
- added R38: 470k, digikey-footprints:0805, F.Cu at (512.8, 87.7)
- added R39: 470k, digikey-footprints:0805, F.Cu at (542.8, 63.7)
- added R4: 470k, digikey-footprints:0805, F.Cu at (438.3, 129.0)
- added R40: 470k, digikey-footprints:0805, F.Cu at (538.5, 63.7)
- added R41: 1MEG, digikey-footprints:0805, F.Cu at (504.5, 96.9)
- added R42: 500k, digikey-footprints:0805, F.Cu at (529.5, 77.6)
- added R43: 1MEG, digikey-footprints:0805, F.Cu at (534.2, 61.9)
- added R44: 500k, digikey-footprints:0805, F.Cu at (519.7, 81.9)
- added R45: 1MEG, digikey-footprints:0805, F.Cu at (534.2, 67.7)
- added R46: 500k, digikey-footprints:0805, F.Cu at (515.5, 81.9)
- added R47: 1MEG, digikey-footprints:0805, F.Cu at (542.6, 57.9)
- added R48: 500k, digikey-footprints:0805, F.Cu at (542.8, 69.5)
- added R49: 22k, digikey-footprints:0805, F.Cu at (525.2, 77.6)
- added R5: 470k, digikey-footprints:0805, F.Cu at (446.8, 122.4)
- added R50: 22k, digikey-footprints:0805, F.Cu at (538.5, 69.5)
- added R51: 22k, digikey-footprints:0805, F.Cu at (528.2, 83.5)
- added R52: 22k, digikey-footprints:0805, F.Cu at (547.0, 63.7)
- added R53: 1MEG, digikey-footprints:0805, F.Cu at (533.8, 79.4)
- added R54: 1MEG, digikey-footprints:0805, F.Cu at (517.1, 93.6)
- added R55: 1MEG, digikey-footprints:0805, F.Cu at (547.0, 57.9)
- added R56: 1MEG, digikey-footprints:0805, F.Cu at (542.5, 75.4)
- added R57: 1MEG, digikey-footprints:0805, F.Cu at (532.6, 85.3)
- added R58: 1MEG, digikey-footprints:0805, F.Cu at (538.2, 81.2)
- added R59: 1MEG, digikey-footprints:0805, F.Cu at (521.5, 89.3)
- added R6: 470k, digikey-footprints:0805, F.Cu at (419.7, 148.8)
- added R60: 1MEG, digikey-footprints:0805, F.Cu at (542.6, 52.0)
- added R61: 470k, digikey-footprints:0805, F.Cu at (546.9, 52.0)
- added R62: 470k, digikey-footprints:0805, F.Cu at (525.4, 71.8)
- added R63: 470k, digikey-footprints:0805, F.Cu at (524.0, 83.5)
- added R64: 470k, digikey-footprints:0805, F.Cu at (533.9, 73.6)
- added R65: 10k, digikey-footprints:0805, F.Cu at (387.7, 172.6)
- added R66: 10k, digikey-footprints:0805, F.Cu at (400.4, 172.6)
- added R67: 10k, digikey-footprints:0805, F.Cu at (396.9, 178.5)
- added R68: 10k, digikey-footprints:0805, F.Cu at (401.2, 178.5)
- added R69: 470k, digikey-footprints:0805, F.Cu at (396.2, 172.6)
- added R7: 470k, digikey-footprints:0805, F.Cu at (442.5, 123.2)
- added R70: 10k, digikey-footprints:0805, F.Cu at (387.7, 178.5)
- added R71: 10k, digikey-footprints:0805, F.Cu at (391.9, 172.6)
- added R72: 10k, digikey-footprints:0805, F.Cu at (504.3, 152.0)
- added R73: 10k, digikey-footprints:0805, F.Cu at (508.6, 152.0)
- added R74: 470k, digikey-footprints:0805, F.Cu at (522.3, 144.6)
- added R75: 10k, digikey-footprints:0805, F.Cu at (512.8, 153.3)
- added R76: 470, digikey-footprints:0805, F.Cu at (526.5, 144.6)
- added R77: 2.2k, digikey-footprints:0805, F.Cu at (517.1, 153.3)
- added R78: 860, digikey-footprints:0805, F.Cu at (521.3, 153.3)
- added R79: 470k, digikey-footprints:0805, F.Cu at (458.9, 151.1)
- added R8: 470k, digikey-footprints:0805, F.Cu at (434.0, 132.3)
- added R80: 100k, digikey-footprints:0805, F.Cu at (525.6, 150.4)
- added R81: 470k, digikey-footprints:0805, F.Cu at (543.3, 134.6)
- added R82: 470k, digikey-footprints:0805, F.Cu at (495.8, 150.8)
- added R83: 10k, digikey-footprints:0805, F.Cu at (546.8, 152.1)
- added R84: 10k, digikey-footprints:0805, F.Cu at (542.6, 152.1)
- added R85: 10k, digikey-footprints:0805, F.Cu at (538.3, 152.1)
- added R86: 10k, digikey-footprints:0805, F.Cu at (543.5, 146.3)
- added R87: 470k, digikey-footprints:0805, F.Cu at (539.3, 146.3)
- added R88: 470k, digikey-footprints:0805, F.Cu at (534.1, 151.6)
- added R89: 10k, digikey-footprints:0805, F.Cu at (545.4, 140.4)
- added R9: 470k, digikey-footprints:0805, F.Cu at (415.4, 148.8)
- added R90: 10k, digikey-footprints:0805, F.Cu at (541.2, 140.4)
- added R91: 10k, digikey-footprints:0805, F.Cu at (535.0, 145.8)
- added R92: 10k, digikey-footprints:0805, F.Cu at (529.8, 151.6)
- added R93: 1MEG, digikey-footprints:0805, F.Cu at (109.2, 161.7)
- added R94: R, digikey-footprints:0805, F.Cu at (367.2, 96.5)
- added R95: R, digikey-footprints:0805, F.Cu at (371.4, 96.5)
- added R96: R, digikey-footprints:0805, F.Cu at (443.2, 52.0)
- added R97: R, digikey-footprints:0805, F.Cu at (447.4, 52.0)
- added R98: R, digikey-footprints:0805, F.Cu at (441.8, 69.5)
- added R99: R, digikey-footprints:0805, F.Cu at (443.2, 57.9)
- added RV1: 100k-S, Potentiometers:Potentiometer_Bourns_PTV09A-1_Horizontal, F.Cu at (121.9, 35.6)
- added RV10: 10kB, Potentiometers:Potentiometer_Bourns_PTV09A-1_Horizontal, F.Cu at (137.2, 53.3)
- added RV11: 10kB, Potentiometers:Potentiometer_Bourns_PTV09A-1_Horizontal, F.Cu at (35.6, 53.3)
- added RV12: 10kA, Potentiometers:Potentiometer_Bourns_PTV09A-1_Horizontal, F.Cu at (121.9, 53.3)
- added RV13: 10kA, Potentiometers:Potentiometer_Bourns_PTV09A-1_Horizontal, F.Cu at (20.3, 53.3)
- added RV14: 10kB, Potentiometers:Potentiometer_Bourns_PTV09A-1_Horizontal, F.Cu at (86.4, 53.3)
- added RV15: 10kB, Potentiometers:Potentiometer_Bourns_PTV09A-1_Horizontal, F.Cu at (188.0, 55.9)
- added RV16: 10kA, Potentiometers:Potentiometer_Bourns_PTV09A-1_Horizontal, F.Cu at (71.1, 53.3)
- added RV17: 10kA, Potentiometers:Potentiometer_Bourns_PTV09A-1_Horizontal, F.Cu at (172.7, 55.9)
- added RV18: 20kA, Potentiometers:Potentiometer_Bourns_PTV09A-1_Horizontal, F.Cu at (27.9, 17.8)
- added RV19: 20kA, Potentiometers:Potentiometer_Bourns_PTV09A-1_Horizontal, F.Cu at (78.7, 17.8)
- added RV2: 100k-S, Potentiometers:Potentiometer_Bourns_PTV09A-1_Horizontal, F.Cu at (20.3, 35.6)
- added RV20: 20kA, Potentiometers:Potentiometer_Bourns_PTV09A-1_Horizontal, F.Cu at (129.5, 17.8)
- added RV21: 20kA, Potentiometers:Potentiometer_Bourns_PTV09A-1_Horizontal, F.Cu at (180.3, 17.8)
- added RV22: 20kA, Potentiometers:Potentiometer_Bourns_PTV09A-1_Horizontal, F.Cu at (35.6, 35.6)
- added RV23: 20kA, Potentiometers:Potentiometer_Bourns_PTV09A-1_Horizontal, F.Cu at (86.4, 35.6)
- added RV24: 20kA, Potentiometers:Potentiometer_Bourns_PTV09A-1_Horizontal, F.Cu at (137.2, 35.6)
- added RV25: 20kA, Potentiometers:Potentiometer_Bourns_PTV09A-1_Horizontal, F.Cu at (188.0, 35.6)
- added RV26: 20kB, Potentiometers:Potentiometer_Bourns_PTV09A-1_Horizontal, F.Cu at (27.9, 71.1)
- added RV27: 20kB, Potentiometers:Potentiometer_Bourns_PTV09A-1_Horizontal, F.Cu at (78.7, 71.1)
- added RV28: 20kB, Potentiometers:Potentiometer_Bourns_PTV09A-1_Horizontal, F.Cu at (129.5, 71.1)
- added RV29: 20kB, Potentiometers:Potentiometer_Bourns_PTV09A-1_Horizontal, F.Cu at (180.3, 73.7)
- added RV3: 100k-S, Potentiometers:Potentiometer_Bourns_PTV09A-1_Horizontal, F.Cu at (71.1, 35.6)
- added RV4: 100k-S, Potentiometers:Potentiometer_Bourns_PTV09A-1_Horizontal, F.Cu at (172.7, 35.6)
- added RV5: 100k, Potentiometers:Potentiometer_Bourns_PTV09A-1_Horizontal, F.Cu at (27.9, 88.9)
- added RV6: 100k, Potentiometers:Potentiometer_Bourns_PTV09A-1_Horizontal, F.Cu at (78.7, 88.9)
- added RV7: 100k, Potentiometers:Potentiometer_Bourns_PTV09A-1_Horizontal, F.Cu at (129.5, 88.9)
- added RV8: 100k, Potentiometers:Potentiometer_Bourns_PTV09A-1_Horizontal, F.Cu at (180.3, 91.4)
- added RV9: 10kA, Potentiometers:Potentiometer_Bourns_PTV09A-1_Horizontal, F.Cu at (520.6, 115.8)
- added SW1: SW_DPDT_x2, SparkFun-Electromechanical:SWITCHE-DPDT, F.Cu at (465.7, 109.1)
- added U1: TL074, digikey-footprints:SOIC-14_W3.9mm, F.Cu at (228.2, 120.3)
- added U2: TL074, digikey-footprints:SOIC-14_W3.9mm, F.Cu at (230.5, 137.1)
- added U3: TL074, digikey-footprints:SOIC-14_W3.9mm, F.Cu at (390.5, 127.8)
- added U4: TL074, digikey-footprints:SOIC-14_W3.9mm, F.Cu at (480.6, -19.7)
- added U5: LD1117S33CTR, digikey-footprints:SOT-223, F.Cu at (459.1, -22.9)
- added U6: TL074, digikey-footprints:SOIC-14_W3.9mm, F.Cu at (510.0, 67.9)
- added U7: TL074, digikey-footprints:Humidity_SHT15, F.Cu at (364.8, 175.5)
- added U8: TL074, digikey-footprints:SMD-5-6_R_3.83x2.79mm, F.Cu at (544.8, 109.4)
- added U9: CY8C4246AZI-L445, digikey-footprints:LQFP-64_10x10mm, F.Cu at (99.1, 160.0)
- added Y1: Crystal, Crystals:Crystal_SMD_HC49-SD_HandSoldering, F.Cu at (114.2, 161.7)
- Q1: value Q_PJFET_DGS -> MMBFJ177
- moved Q1 371.7 mm to (519.0, 75.5)
Connections:
- Q1 pad 2: Net-(Q1-Pad2) -> GND
Other:
- board outline added: 203.2 x 101.6 mm

Commit message: fix annotation and footprints for multi-part op amps.
Parts:
- removed U9: CY8C4246AZI-L445, digikey-footprints:LQFP-64_10x10mm
- U7: value TL074 -> CY8C4246AZI-L445; footprint digikey-footprints:Humidity_SHT15 -> digikey-footprints:LQFP-64_10x10mm
- moved C31 539.5 mm to (-36.2, 36.2), turned to 270 degrees
- moved C30 531.5 mm to (-36.2, 27.3), turned to 90 degrees
- moved D1 516.8 mm to (-45.7, 26.7), turned to 180 degrees
- moved U5 506.4 mm to (-43.8, 36.2), turned to 90 degrees
- moved J1 495.9 mm to (-38.7, 19.7), turned to 270 degrees
- moved RV9 417.9 mm to (104.1, 81.3), turned to 90 degrees
- moved SW1 364.8 mm to (101.6, 86.4)
- moved U4 363.7 mm to (121.9, -80.0)
- moved C29 342.3 mm to (151.1, -76.2), turned to 270 degrees
- moved R34 333.0 mm to (152.4, -83.8), turned to 90 degrees
- moved R33 329.2 mm to (149.9, -83.8), turned to 270 degrees
- moved U7 266.3 mm to (99.1, 158.8), turned to 270 degrees
- moved U1 235.9 mm to (429.3, 243.8)
- moved U2 212.3 mm to (414.0, 243.8)
- moved C7 132.3 mm to (417.8, 252.7), turned to 270 degrees
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Connections:
- U1 pad 1: Net-(C10-Pad1) -> Net-(C13-Pad1)
- U1 pad 10: Net-(C9-Pad1) -> Net-(C23-Pad1)
- U1 pad 12: Net-(C4-Pad1) -> Net-(C24-Pad1)
- U1 pad 13: Net-(C13-Pad1) -> Net-(C25-Pad1)
- U1 pad 14: Net-(C13-Pad1) -> Net-(C25-Pad1)
- U1 pad 2: Net-(C10-Pad1) -> Net-(C13-Pad1)
- U1 pad 3: Net-(C5-Pad1) -> Net-(C4-Pad1)
- U1 pad 5: Net-(C7-Pad1) -> Net-(C5-Pad1)
- U1 pad 6: Net-(C11-Pad1) -> Net-(C10-Pad1)
- U1 pad 7: Net-(C11-Pad1) -> Net-(C10-Pad1)
- U1 pad 8: Net-(C12-Pad1) -> Net-(C26-Pad1)
- U1 pad 9: Net-(C12-Pad1) -> Net-(C26-Pad1)
- U2 pad 10: Net-(R16-Pad1) -> Net-(C8-Pad1)
- U2 pad 12: Net-(R17-Pad1) -> Net-(C9-Pad1)
- U2 pad 13: Net-(C17-Pad2) -> Net-(C12-Pad1)
- U2 pad 14: Net-(C17-Pad1) -> Net-(C12-Pad1)
- U2 pad 5: Net-(C8-Pad1) -> Net-(C7-Pad1)
- U2 pad 6: Net-(C15-Pad1) -> Net-(C11-Pad1)
- U2 pad 7: Net-(C15-Pad1) -> Net-(C11-Pad1)
- U2 pad 8: Net-(C16-Pad1) -> Net-(C15-Pad1)
- U2 pad 9: Net-(C16-Pad2) -> Net-(C15-Pad1)
- U3 pad 1: Net-(C18-Pad1) -> Net-(C17-Pad1)
- U3 pad 10: Net-(C23-Pad1) -> Net-(R16-Pad1)
- U3 pad 2: Net-(C18-Pad2) -> Net-(C17-Pad2)
- U3 pad 3: Net-(R18-Pad1) -> Net-(R17-Pad1)
- U3 pad 5: Net-(C24-Pad1) -> Net-(R18-Pad1)
- U3 pad 6: Net-(C25-Pad1) -> Net-(C18-Pad2)
- U3 pad 7: Net-(C25-Pad1) -> Net-(C18-Pad1)
- U3 pad 8: Net-(C26-Pad1) -> Net-(C16-Pad1)
- U3 pad 9: Net-(C26-Pad1) -> Net-(C16-Pad2)
- U4 pad 1: VREF -> Net-(R75-Pad1)
- U4 pad 10: (no net) -> Net-(R69-Pad1)
- U4 pad 12: (no net) -> Net-(C29-Pad1)
- U4 pad 13: (no net) -> VREF
- U4 pad 14: (no net) -> VREF
- U4 pad 2: VREF -> Net-(R74-Pad1)
- U4 pad 3: Net-(C29-Pad1) -> Net-(R75-Pad2)
- U4 pad 5: (no net) -> Net-(R79-Pad1)
- U4 pad 6: (no net) -> Net-(C58-Pad1)
- U4 pad 7: (no net) -> Net-(C58-Pad2)
- U4 pad 8: (no net) -> Net-(C56-Pad1)
- U4 pad 9: (no net) -> Net-(C56-Pad2)
- U7 pad 1: Net-(C56-Pad1) -> /Microcontroller/osc1_speed
- U7 pad 2: Net-(C56-Pad2) -> /Microcontroller/osc4_pwm_wiper
- U7 pad 3: Net-(R69-Pad1) -> /Microcontroller/osc4_freq_wiper
- U7 pad 4: GND -> /Microcontroller/osc3_pwm_wiper
- U7 pad 5: Net-(R75-Pad2) -> /Microcontroller/osc3_freq_wiper
- U7 pad 6: Net-(R74-Pad1) -> /Microcontroller/osc2_pwm_wiper
- U7 pad 7: Net-(R75-Pad1) -> /Microcontroller/osc2_freq_wiper
- U7 pad 8: +15V -> /Microcontroller/osc1_pwm_wiper

Commit message: loosely organize components into groups based on their functionality
Parts:
- removed U8: TL074, digikey-footprints:SMD-5-6_R_3.83x2.79mm
- C29, C30, C31, C52, C53, C54, C55, C56, C57, C58, C59, C60, C61, C62, C63, C64, C65, C66, C67, C68, C69, C70, C71, C72, C73, D1, D2, J3, Q5, Q6, Q7, Q8, R33, R34, R65, R66, R67, R68, R69, R70, R71, R72, R73, R74, R75, R76, R77, R78, R79, R80, R81, R82, R83, R84, R85, R86, R87, R88, R89, R90, R91, R92, R93, U4, U5, U7, Y1: moved to B.Cu
- moved R86 540.9 mm to (27.1, -14.8)
- moved Q6 540.1 mm to (27.9, -35.6)
- moved R85 534.5 mm to (30.3, -14.2)
- moved C61 523.5 mm to (32.9, -27.2)
- moved C65 497.5 mm to (20.9, -25.2)
- moved R89 493.5 mm to (78.8, -20.3)
- moved R90 493.5 mm to (74.6, -20.3)
- moved R82 492.4 mm to (33.9, -19.8)
- moved Q7 490.5 mm to (73.7, -25.4)
- moved R87 490.3 mm to (79.4, -23.9)
- moved C70 482.8 mm to (76.4, -15.5)
- moved C68 476.3 mm to (81.0, -10.9)
- moved C66 472.4 mm to (76.8, -11.1)
- moved C63 468.2 mm to (25.9, -16.4)
- moved C58 449.6 mm to (96.5, 35.6), turned to 180 degrees
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
Commit message: component placement mostly finalized
Parts:
- C1, C10, C11, C12, C13, C14, C15, C16, C17, C18, C19, C2, C20, C21, C22, C23, C24, C25, C26, C27, C28, C3, C32, C33, C34, C35, C36, C37, C38, C39, C4, C40, C41, C42, C43, C44, C45, C46, C47, C48, C49, C5, C50, C51, C6, C7, C8, C9, Q1, Q2, Q3, Q4, R1, R10, R100, R101, R102, R103, R104, R105, R11, R12, R13, R14, R15, R16, R17, R18, R19, R2, R20, R21, R22, R23, R24, R25, R26, R27, R28, R29, R3, R30, R31, R32, R35, R36, R37, R38, R39, R4, R40, R41, R42, R43, R44, R45, R46, R47, R48, R49, R5, R50, R51, R52, R53, R54, R55, R56, R57, R58, R59, R6, R60, R61, R62, R63, R64, R7, R8, R9, R94, R95, R96, R97, R98, R99, U1, U2, U3, U6: moved to B.Cu
- moved R14 480.2 mm to (-1.91, -54.0)
- moved R15 442.8 mm to (41.9, -54.0), turned to 180 degrees
- moved R13 438.2 mm to (-1.91, -48.3)
- moved R24 416.9 mm to (84.8, -75.7), turned to 90 degrees
- moved R2 416.4 mm to (20.3, -37.5), turned to 180 degrees
- moved C21 413.7 mm to (90.4, -74.7), turned to 180 degrees
- moved C11 410.6 mm to (10.2, -48.3), turned to 180 degrees
- moved C6 410.3 mm to (23.5, -42.5), turned to 270 degrees
- moved C18 409.3 mm to (97.0, -70.1), turned to 0 degrees
- moved R21 409.0 mm to (97.0, -72.1), turned to 0 degrees
- moved R18 404.6 mm to (100.1, -71.1), turned to 270 degrees
- moved R5 403.4 mm to (12.7, -43.2)
- moved C2 399.7 mm to (31.8, -41.9), turned to 90 degrees
- moved R8 399.7 mm to (27.9, -42.5), turned to 90 degrees
- moved R16 399.3 mm to (100.1, -83.3), turned to 90 degrees
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
Commit message: MCU bypass capacitor routing complete
Parts:
- added C74: 1uF, Capacitors_SMD:C_0805, B.Cu at (63.5, 85.1)
- added C75: 1uF, Capacitors_SMD:C_0805, B.Cu at (52.6, 73.7)
- added C76: 0.1uF, Capacitors_SMD:C_0805, B.Cu at (61.5, 85.1)
- added C77: 0.1uF, Capacitors_SMD:C_0805, B.Cu at (52.6, 75.7)
- added C78: 1uF, Capacitors_SMD:C_0805, B.Cu at (48.8, 73.7)
- added C79: 0.1uF, Capacitors_SMD:C_0805, B.Cu at (53.1, 92.7)
- added C80: 0.1uF, Capacitors_SMD:C_0805, B.Cu at (48.8, 75.7)
- added C81: 1uF, Capacitors_SMD:C_0805, B.Cu at (53.1, 94.7)
- added C82: 1uF, Capacitors_SMD:C_0805, B.Cu at (44.5, 79.0)
- added R106: R, digikey-footprints:0805, B.Cu at (44.5, 74.9)
- added R107: R, digikey-footprints:0805, F.Cu at (3.30, 47.2)
- moved C43 186.1 mm to (256.5, 62.6)
- moved R60 186.1 mm to (256.5, 65.2)
- moved C32 186.1 mm to (248.9, 103.3)
- moved C33 186.1 mm to (240.0, 103.3)
- moved C34 186.1 mm to (232.4, 46.1)
- moved C35 186.1 mm to (241.3, 46.1)
- moved C36 186.1 mm to (250.2, 46.1)
- moved C37 186.1 mm to (259.1, 46.1)
- moved C38 186.1 mm to (231.1, 103.3)
- moved C39 186.1 mm to (222.2, 103.3)
- moved C40 186.1 mm to (249.6, 92.5)
- moved C41 186.1 mm to (238.1, 87.4)
- moved C42 186.1 mm to (247.0, 55.6)
- moved C44 186.1 mm to (247.7, 82.3)
- moved C45 186.1 mm to (241.9, 82.3)
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Connections:
- U7 pad 10: Net-(U7-Pad10) -> GNDD
- U7 pad 11: Net-(U7-Pad11) -> +3V3
- U7 pad 17: Net-(U7-Pad17) -> GNDD
- U7 pad 26: Net-(U7-Pad26) -> +3V3
- U7 pad 49: Net-(U7-Pad49) -> GNDD
- U7 pad 50: Net-(U7-Pad50) -> +3V3
- U7 pad 56: Net-(U7-Pad56) -> +3V3
- U7 pad 57: Net-(U7-Pad57) -> GNDD
Routing:
- net GNDD: track 0.00 -> 165.6 mm, vias 0 -> 3
- net +3V3: track 0.00 -> 157.6 mm, vias 0 -> 1
- net Net-(C73-Pad1): track 0.00 -> 17.9 mm
- net Net-(C72-Pad1): track 0.00 -> 14.4 mm
- net /Microcontroller/SDAT: track 0.00 -> 12.9 mm, vias 0 -> 1
- net /Microcontroller/SCLK: track 0.00 -> 11.7 mm, vias 0 -> 1
- net /Microcontroller/XRES: track 0.00 -> 9.58 mm
- net GND: track 0.00 -> 5.56 mm, vias 0 -> 1
- net +15V: track 0.00 -> 4.95 mm
- net Net-(R98-Pad2): track 0.00 -> 3.73 mm
- net Net-(R94-Pad2): track 0.00 -> 3.43 mm
- net Net-(C82-Pad1): track 0.00 -> 2.51 mm
Other:
- net class PWR added: clearance 0.3, trace_width 0.75, via_dia 0.8, via_drill 0.5

Commit message: gettin' there. WIP
Parts:
- R107: moved to B.Cu
- moved R72 113.1 mm to (93.0, 121.5)
- moved R73 113.1 mm to (95.0, 121.5)
- moved J2 92.8 mm to (92.8, 96.2)
- moved R71 79.5 mm to (85.8, 97.2), turned to 0 degrees
- moved C53 75.2 mm to (115.2, 76.2), turned to 0 degrees
- moved C52 74.9 mm to (115.2, 82.0), turned to 0 degrees
- moved C57 74.3 mm to (87.0, 91.5), turned to 270 degrees
- moved R65 69.8 mm to (109.5, 78.7), turned to 270 degrees
- moved C17 63.8 mm to (96.6, 5.91), turned to 0 degrees
- moved C18 63.6 mm to (104.7, 5.91), turned to 180 degrees
- moved R23 63.1 mm to (85.0, 9.50)
- moved R66 63.0 mm to (109.8, 72.2), turned to 270 degrees
- moved R17 61.2 mm to (99.6, 6.93), turned to 90 degrees
- moved R18 61.2 mm to (101.7, 6.93), turned to 90 degrees
- moved R24 60.8 mm to (116.9, 11.5), turned to 270 degrees
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Connections:
- U7 pad 2: /Microcontroller/osc4_pwm_wiper -> /Microcontroller/osc1_freq_wiper
- U7 pad 3: /Microcontroller/osc4_freq_wiper -> /Microcontroller/osc1_pwm_wiper
- U7 pad 4: /Microcontroller/osc3_pwm_wiper -> /Microcontroller/osc2_freq_wiper
- U7 pad 5: /Microcontroller/osc3_freq_wiper -> /Microcontroller/osc2_pwm_wiper
- U7 pad 6: /Microcontroller/osc2_pwm_wiper -> /Microcontroller/osc3_freq_wiper
- U7 pad 7: /Microcontroller/osc2_freq_wiper -> /Microcontroller/osc3_pwm_wiper
- U7 pad 8: /Microcontroller/osc1_pwm_wiper -> /Microcontroller/osc4_freq_wiper
- U7 pad 9: /Microcontroller/osc1_freq_wiper -> /Microcontroller/osc4_pwm_wiper
Routing:
- net +3V3: track 157.6 -> 614.0 mm, vias 1 -> 5
- net /Microcontroller/osc4_pwm_wiper: track 0.00 -> 169.3 mm, vias 0 -> 1
- net /Microcontroller/osc4_freq_wiper: track 0.00 -> 167.9 mm, vias 0 -> 1
- net /Microcontroller/osc4_speed: track 0.00 -> 148.3 mm, vias 0 -> 1
- net Net-(C18-Pad2): track 0.00 -> 120.5 mm
- net /Microcontroller/osc3_pwm_wiper: track 0.00 -> 116.6 mm, vias 0 -> 1
- net /Microcontroller/osc3_freq_wiper: track 0.00 -> 116.1 mm, vias 0 -> 1
- net /Microcontroller/osc3_speed: track 0.00 -> 97.1 mm, vias 0 -> 1
- net /Microcontroller/osc2_freq_wiper: track 0.00 -> 95.0 mm, vias 0 -> 1
- net /Filters/osc2: track 0.00 -> 91.4 mm, vias 0 -> 2
- net Net-(C17-Pad2): track 0.00 -> 74.7 mm
- net Net-(C13-Pad2): track 0.00 -> 72.9 mm, vias 0 -> 2
- net /Microcontroller/osc1_freq_wiper: track 0.00 -> 72.7 mm, vias 0 -> 1
- net /Microcontroller/osc2_pwm_wiper: track 0.00 -> 70.0 mm, vias 0 -> 1
- net Net-(C14-Pad2): track 0.00 -> 63.9 mm, vias 0 -> 1
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- added copper zone on B.Cu, net GND
- added copper zone on F.Cu, net GND

Commit message: complete initial PCB layout. CapSense buttons still not done, but everything else should be there. I had to increase to a 4-layer board to keep the dimensions 8"x4".
Parts:
- D1: value D -> D_Schottky; footprint digikey-footprints:TO-252-3 -> Diodes_SMD:D_SMB
- moved C48 229.3 mm to (27.2, 94.0), turned to 180 degrees
- moved C49 170.6 mm to (66.0, 86.0), turned to 270 degrees
- moved R35 161.4 mm to (58.8, 42.8), turned to 90 degrees
- moved R36 159.2 mm to (56.6, 42.8), turned to 270 degrees
- moved C33 146.1 mm to (94.0, 97.0), turned to 180 degrees
- moved R42 140.9 mm to (101.0, 98.0), turned to 90 degrees
- moved C35 129.5 mm to (122.1, 96.7), turned to 180 degrees
- moved C50 121.6 mm to (116.0, 88.0), turned to 0 degrees
- moved R46 118.4 mm to (129.0, 96.0), turned to 270 degrees
- moved R64 114.7 mm to (138.0, 80.0), turned to 90 degrees
- moved C39 114.4 mm to (108.0, 97.0), turned to 180 degrees
- moved R41 113.6 mm to (133.5, 97.0), turned to 90 degrees
- moved R44 109.2 mm to (115.0, 98.0), turned to 90 degrees
- moved C32 108.7 mm to (140.5, 96.0), turned to 0 degrees
- moved C40 108.1 mm to (141.6, 88.5)
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Connections:
- C37 pad 2: Net-(C37-Pad2) -> /Microcontroller/envelope_pwm_4
- U1 pad 11: GND -> +15V
- U1 pad 2: Net-(C13-Pad1) -> Net-(C4-Pad1)
- U1 pad 3: Net-(C4-Pad1) -> Net-(C13-Pad1)
- U1 pad 4: +15V -> GND
Routing:
- net +15V: track 4.95 -> 480.0 mm, vias 0 -> 12
- net /Envelope/lfo_bias: track 0.00 -> 251.9 mm, vias 0 -> 4
- net /LFO Modulation and Routing/bias: track 0.00 -> 247.9 mm, vias 0 -> 7
- net /Envelope/lfo1: track 0.00 -> 198.0 mm, vias 0 -> 1
- net /LFO Modulation and Routing/main_lfo: track 0.00 -> 185.8 mm, vias 0 -> 5
- net /Filters/osc4: track 3.76 -> 181.4 mm, vias 0 -> 2
- net /Filters/filter_out_4: track 4.21 -> 163.5 mm, vias 0 -> 2
- net /Filters/osc3: track 3.76 -> 150.1 mm, vias 0 -> 2
- net Net-(C48-Pad1): track 0.00 -> 138.2 mm, vias 0 -> 2
- net /Microcontroller/envelope_pwm_4: track 0.00 -> 136.7 mm, vias 0 -> 2
- net /Filters/filter_out_1: track 4.37 -> 115.5 mm, vias 0 -> 4
- net /Envelope/lfo2: track 0.00 -> 107.9 mm, vias 0 -> 3
- net /Envelope/env_out_1: track 0.00 -> 106.0 mm, vias 0 -> 1
- net Net-(R47-Pad1): track 0.00 -> 104.3 mm, vias 0 -> 2
- net Net-(C49-Pad1): track 0.00 -> 103.6 mm, vias 0 -> 2
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- added copper zone on In2.Cu, net GND
- added copper zone on In1.Cu, net VREF
Other:
- copper layers 2 -> 4

Commit message: complete PCB v1, no DRC errors.
Parts:
- added J4: Capsense_0, Cypress_capsense:Capsense_button, F.Cu at (12.7, 81.3)
- added J5: Capsense_1, Cypress_capsense:Capsense_button, F.Cu at (12.7, 73.7)
- added J6: Capsense_2, Cypress_capsense:Capsense_button, F.Cu at (12.7, 66.0)
- added J7: Capsense_3, Cypress_capsense:Capsense_button, F.Cu at (12.7, 58.7)
Routing:
- net GND: track 34.8 -> 366.2 mm, vias 9 -> 27
- net VREF: track 62.4 -> 195.3 mm, vias 17 -> 25
- net Net-(J7-Pad1): track 0.00 -> 67.4 mm, vias 0 -> 3
- net Net-(J6-Pad1): track 0.00 -> 61.8 mm, vias 0 -> 3
- net Net-(J5-Pad1): track 0.00 -> 55.9 mm, vias 0 -> 3
- net Net-(J4-Pad1): track 0.00 -> 50.4 mm, vias 0 -> 3
- net +3V3: track 619.9 -> 644.9 mm, vias 5 -> 7
- net Net-(C69-Pad2): track 43.7 -> 52.3 mm, vias 0 -> 2
- net Net-(C67-Pad1): track 0.00 -> 8.29 mm
- net /Filters/filter_out_4: track 163.5 -> 158.9 mm
- net Net-(C69-Pad1): track 0.00 -> 4.56 mm
- net Net-(C46-Pad1): track 4.08 -> 8.29 mm
- net /Microcontroller/XRES: track 38.7 -> 42.9 mm
- net Net-(C62-Pad2): track 27.0 -> 31.1 mm
- net +15V: track 480.0 -> 477.5 mm
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