File: Hardware/synth_psoc.kicad_pcb (KiCad board)
At the start: 4 copper layers, 203.2 x 101.6 mm, 244 parts, among them J1 Barrel_Jack, J2 Audio-Jack-2_Switch, J3 SWD_programming, J4 Capsense_0, J5 Capsense_1, J6 Capsense_2, J7 Capsense_3, Q1 MMBFJ177, Q2 MMBFJ177, Q3 MMBFJ177, Q4 MMBFJ177, Q5 2N3904, Q6 2N3904, Q7 2N3904, Q8 2N3904, SW1 SW_DPDT_x2, U1 TL074, U2 TL074, U3 TL074, U4 TL074, U5 LD1117S33CTR, U6 TL074, U7 CY8C4246AZI-L445, Y1 Crystal

Commit message: as built v1 boards, 2019-01-16 with gerber outputs
Parts:
- moved R2 1.40 mm to (47.8, 28.4)
Routing:
- net Net-(C2-Pad1): track 13.7 -> 14.7 mm

Commit message: begin PCB v2 layout. fix ref designators, associate footprints on new components, create new PCB file, import components.
Parts:
- added C83: 1uF, Capacitors_SMD:CP_Elec_4x4.5, F.Cu at (299.7, 112.3)
- added C84: 0.1uF, digikey-footprints:0805, F.Cu at (269.5, 147.4)
- added C85: 0.1uF, digikey-footprints:0805, F.Cu at (265.6, 153.2)
- added C86: 1uF, Capacitors_SMD:CP_Elec_4x4.5, F.Cu at (275.7, 129.7)
- added C87: 22pF, digikey-footprints:0805, F.Cu at (307.4, 108.9)
- added C88: 1uF, Capacitors_SMD:CP_Elec_4x4.5, F.Cu at (266.6, 139.9)
- added C89: 2.2nF, digikey-footprints:0805, F.Cu at (276.7, 137.1)
- added C90: CP1_Small, Capacitors_SMD:CP_Elec_5x5.7, F.Cu at (237.5, 129.1)
- added C91: CP1_Small, Capacitors_SMD:CP_Elec_5x5.7, F.Cu at (207.0, 149.4)
- added C92: CP1_Small, Capacitors_SMD:CP_Elec_5x5.7, F.Cu at (198.6, 149.4)
- added C93: CP1_Small, Capacitors_SMD:CP_Elec_5x5.7, F.Cu at (198.6, 97.5)
- added R108: R, digikey-footprints:0805, F.Cu at (315.9, 103.7)
- added R109: R, digikey-footprints:0805, F.Cu at (294.9, 119.8)
- added R110: R, digikey-footprints:0805, F.Cu at (311.7, 103.7)
- added R111: R, digikey-footprints:0805, F.Cu at (315.2, 86.2)
- added R112: R, digikey-footprints:0805, F.Cu at (290.2, 130.0)
- added R113: R, digikey-footprints:0805, F.Cu at (248.2, 156.3)
- added R114: R, digikey-footprints:0805, F.Cu at (307.4, 103.1)
- added R115: R, digikey-footprints:0805, F.Cu at (252.4, 156.3)
- added R116: R, digikey-footprints:0805, F.Cu at (315.2, 92.1)
- added R117: R, digikey-footprints:0805, F.Cu at (184.6, 156.5)
- added R118: R, digikey-footprints:0805, F.Cu at (315.2, 97.9)
- added RV30: 20kB, Potentiometers:Potentiometer_Bourns_PTV09A-1_Horizontal, F.Cu at (270.7, 94.5)
- added RV31: 20kB, Potentiometers:Potentiometer_Bourns_PTV09A-1_Horizontal, F.Cu at (243.8, 129.9)
- added RV32: 20kB, Potentiometers:Potentiometer_Bourns_PTV09A-1_Horizontal, F.Cu at (219.8, 152.6)
- added RV33: 20kB, Potentiometers:Potentiometer_Bourns_PTV09A-1_Horizontal, F.Cu at (258.6, 111.9)
- added SW10: SW_SPST, SparkFun-Electromechanical:SWITCH-SPDT, F.Cu at (198.9, 134.2)
- added SW11: SW_SPST, SparkFun-Electromechanical:SWITCH-SPDT, F.Cu at (210.9, 134.2)
- added SW12: SW_SPST, SparkFun-Electromechanical:SWITCH-SPDT, F.Cu at (234.9, 113.8)
- added SW13: SW_SPST, SparkFun-Electromechanical:SWITCH-SPDT, F.Cu at (222.9, 113.8)
- added SW2: SW_SPST, SparkFun-Electromechanical:SWITCH-SPDT, F.Cu at (186.9, 123.0)
- added SW3: SW_SPST, SparkFun-Electromechanical:SWITCH-SPDT, F.Cu at (198.9, 113.8)
- added SW4: SW_SPST, SparkFun-Electromechanical:SWITCH-SPDT, F.Cu at (219.8, 93.5)
- added SW5: SW_SPST, SparkFun-Electromechanical:SWITCH-SPDT, F.Cu at (186.9, 102.6)
- added SW6: SW_SPST, SparkFun-Electromechanical:SWITCH-SPDT, F.Cu at (207.8, 93.5)
- added SW7: SW_SPST, SparkFun-Electromechanical:SWITCH-SPDT, F.Cu at (186.9, 143.4)
- added SW8: SW_SPST, SparkFun-Electromechanical:SWITCH-SPDT, F.Cu at (231.8, 93.5)
- added SW9: SW_SPST, SparkFun-Electromechanical:SWITCH-SPDT, F.Cu at (210.9, 113.8)
- added U8: PT2399, digikey-footprints:DIP-16_W7.62mm, F.Cu at (322.3, 87.6)
- C1, C2, C3: value 1uF -> 22uF; footprint Capacitors_SMD:CP_Elec_4x4.5 -> Capacitors_SMD:CP_Elec_5x5.7; moved to F.Cu
- C10, C11, C12, C5, C6, C7, C8, C9: value 22uF -> 10nF; footprint Capacitors_SMD:CP_Elec_5x5.7 -> digikey-footprints:0805; moved to F.Cu
- C13, C14, C15, C22, C4, C44, C45, C46, C47, C52, D1, D2, J3, R1, R100, R101, R102, R103, R104, R105, R106, R107, R2, R26, R3, R35, R36, R41, R43, R45, R61, R62, R66, R67, R68, R73, R75, R88, R9, R93, R94, R95, R96, R97, R98, R99, U1, U2, U3, U4, Y1: moved to F.Cu
- C16: value 100p -> 22uF; footprint digikey-footprints:0805 -> Capacitors_SMD:CP_Elec_5x5.7; moved to F.Cu
- C17: value 100p -> 220uF; footprint digikey-footprints:0805 -> Capacitors_SMD:CP_Elec_8x10; moved to F.Cu
- C18: value 100p -> 0.33uF; moved to F.Cu
- C19, C49, C51, C54: value 22uF -> 0.1uF; footprint Capacitors_SMD:CP_Elec_5x5.7 -> digikey-footprints:0805; moved to F.Cu
- C20, C21, C23: value 22uF -> 1uF; footprint Capacitors_SMD:CP_Elec_5x5.7 -> Capacitors_SMD:CP_Elec_4x4.5; moved to F.Cu
- C24, C25, C26, C28: value 22uF -> 220u; footprint Capacitors_SMD:CP_Elec_5x5.7 -> Capacitors_SMD:CP_Elec_8x10; moved to F.Cu
- C27: value 100p -> 220u; footprint digikey-footprints:0805 -> Capacitors_SMD:CP_Elec_8x10; moved to F.Cu
- C29: value 220uF -> 220u; moved to F.Cu
- C30: value 1uF -> 220u; footprint Capacitors_SMD:CP_Elec_4x4.5 -> Capacitors_SMD:CP_Elec_8x10; moved to F.Cu
- C31: value 4.7uF -> 220u; footprint Capacitors_SMD:CP_Elec_4x5.7 -> Capacitors_SMD:CP_Elec_8x10; moved to F.Cu
- C32, C33, C34, C35: value 220u -> 1nF; footprint Capacitors_SMD:CP_Elec_8x10 -> digikey-footprints:0805; moved to F.Cu
- C36, C37, C38, C39: value 220u -> 22uF; footprint Capacitors_SMD:CP_Elec_8x10 -> Capacitors_SMD:CP_Elec_5x5.7; moved to F.Cu
- C40, C41, C42, C43: value 1nF -> 22uF; footprint digikey-footprints:0805 -> Capacitors_SMD:CP_Elec_5x5.7; moved to F.Cu
- C48, C61: value 22uF -> 100pF; footprint Capacitors_SMD:CP_Elec_5x5.7 -> digikey-footprints:0805; moved to F.Cu
- C50: value 22uF -> 100uF; moved to F.Cu
- C53: value 22uF -> 47uF; footprint Capacitors_SMD:CP_Elec_5x5.7 -> Capacitors_SMD:CP_Elec_4x5.7; moved to F.Cu
- C55: value 22uF -> 560pF; footprint Capacitors_SMD:CP_Elec_5x5.7 -> digikey-footprints:0805; moved to F.Cu
- C56: value 100pF -> 560pF; moved to F.Cu
- C57, C58: value 22uF -> 82nF; footprint Capacitors_SMD:CP_Elec_5x5.7 -> digikey-footprints:0805; moved to F.Cu
- C59: value 220uF -> 3900pF; footprint Capacitors_SMD:CP_Elec_8x10 -> digikey-footprints:0805; moved to F.Cu
- C60: value 22uF -> 3300pF; footprint Capacitors_SMD:CP_Elec_5x5.7 -> digikey-footprints:0805; moved to F.Cu
- C62, C68: value 33nF -> 100pF; moved to F.Cu
- C63: value 33nF -> 4.7uF; footprint digikey-footprints:0805 -> Capacitors_SMD:CP_Elec_4x5.7; moved to F.Cu
- C64: value 22uF -> 0.01uF; footprint Capacitors_SMD:CP_Elec_5x5.7 -> digikey-footprints:0805; moved to F.Cu
- C65: value 220uF -> 4.7uF; footprint Capacitors_SMD:CP_Elec_8x10 -> Capacitors_SMD:CP_Elec_4x5.7; moved to F.Cu
- C66, C67: value 22uF -> 10uF; footprint Capacitors_SMD:CP_Elec_5x5.7 -> Capacitors_SMD:CP_Elec_4x5.7; moved to F.Cu
- C69: value 33nF -> 22uF; footprint digikey-footprints:0805 -> Capacitors_SMD:CP_Elec_5x5.7; moved to F.Cu
- C70, C71: value 22uF -> 220uF; footprint Capacitors_SMD:CP_Elec_5x5.7 -> Capacitors_SMD:CP_Elec_8x10; moved to F.Cu
- C72: value 22pF -> 22uF; footprint digikey-footprints:0805 -> Capacitors_SMD:CP_Elec_5x5.7; moved to F.Cu
- C73: value 22pF -> 220uF; footprint digikey-footprints:0805 -> Capacitors_SMD:CP_Elec_8x10; moved to F.Cu
- C74, C75: value 1uF -> 220uF; footprint Capacitors_SMD:C_0805 -> Capacitors_SMD:CP_Elec_8x10; moved to F.Cu
- C76, C77: value 0.1uF -> 220uF; footprint Capacitors_SMD:C_0805 -> Capacitors_SMD:CP_Elec_8x10; moved to F.Cu
- C78: footprint Capacitors_SMD:C_0805 -> Capacitors_SMD:CP_Elec_4x4.5; moved to F.Cu
- C79: value 0.1uF -> 1uF; footprint Capacitors_SMD:C_0805 -> Capacitors_SMD:CP_Elec_4x4.5; moved to F.Cu
- C80: footprint Capacitors_SMD:C_0805 -> digikey-footprints:0805; moved to F.Cu
- C81: value 1uF -> 0.1uF; footprint Capacitors_SMD:C_0805 -> digikey-footprints:0805; moved to F.Cu
- C82: value 1uF -> 22pF; footprint Capacitors_SMD:C_0805 -> digikey-footprints:0805; moved to F.Cu
- Q1: value MMBFJ177 -> MMBT3904-TP; footprint TO_SOT_Packages_SMD:SOT-23 -> digikey-footprints:SOT-23-3; moved to F.Cu
- Q2, Q3, Q4: value MMBFJ177 -> MMBT3904-TP; moved to F.Cu
- Q5, Q6, Q7, Q8: value 2N3904 -> MMBFJ177; moved to F.Cu
- R10, R11, R12, R86, R89, R90, R91: value 10k -> 470k; moved to F.Cu
- R13, R14, R15, R72, R85: value 10k -> 100k; moved to F.Cu
- R16, R17, R18, R87: value 470k -> 100k; moved to F.Cu
- R19, R20, R21: value 10k -> 1k; moved to F.Cu
- R22: value 100k -> 1k; moved to F.Cu
- R23, R24, R80: value 100k -> 470k; moved to F.Cu
- R25: value 1k -> 470k; moved to F.Cu
- R27, R39, R40: value 470k -> 1MEG; moved to F.Cu
- R28: value 10k -> 500k; moved to F.Cu
- R29, R31: value 10k -> 1MEG; moved to F.Cu
- R30: value 470k -> 500k; moved to F.Cu
- R32, R34: value 100k -> 500k; moved to F.Cu
- R33: value 100k -> 1MEG; moved to F.Cu
- R37, R38: value 470k -> 22k; moved to F.Cu
- R4, R5, R6, R7, R8: value 470k -> 1k; moved to F.Cu
- R42, R44, R46: value 500k -> 1MEG; moved to F.Cu
- R47, R55: value 1MEG -> 470k; moved to F.Cu
- R48: value 500k -> 470k; moved to F.Cu
- R49, R50: value 22k -> 470k; moved to F.Cu
- R51, R52: value 22k -> 10k; moved to F.Cu
- R53, R54, R56, R58, R59, R60: value 1MEG -> 10k; moved to F.Cu
- R57: value 1MEG -> 4.7k; moved to F.Cu
- R63, R64, R69, R74, R79, R81: value 470k -> 10k; moved to F.Cu
- R65, R70: value 10k -> 15k; moved to F.Cu
- R71: value 10k -> 5.6k; moved to F.Cu
- R76: value 470 -> 470k; moved to F.Cu
- R77: value 2.2k -> 4.7k; moved to F.Cu
- R78: value 860 -> 10k; moved to F.Cu
- R82: value 470k -> 470; moved to F.Cu
- R83: value 10k -> 2.2k; moved to F.Cu
- R84: value 10k -> 860; moved to F.Cu
- R92: value 10k -> R; moved to F.Cu
- RV1, RV2, RV3, RV4: value 100k-S -> POT_Dual; footprint Potentiometers:Potentiometer_Bourns_PTV09A-1_Horizontal -> Potentiometers:Potentiometer_Trimmer-EVM3E
- RV10, RV11: value 10kB -> 100kA
- RV12, RV9: value 10kA -> 100kA
- RV13: value 10kA -> 20kA
- RV14: value 10kB -> 20k
- RV15: value 10kB -> 50kA
- RV16: value 10kA -> 50kA
- RV18, RV19, RV20, RV21: value 20kA -> 10kA
- RV26, RV27, RV28, RV29: value 20kB -> 20kA
- RV5, RV6, RV7, RV8: value 100k -> POT_TRIM; footprint Potentiometers:Potentiometer_Bourns_PTV09A-1_Horizontal -> Potentiometers:Potentiometer_Trimmer-EVM3E
- SW1: footprint SparkFun-Electromechanical:SWITCHE-DPDT -> SparkFun-Electromechanical:SWITCH-SPDT
- U5: value LD1117S33CTR -> TL074; footprint digikey-footprints:SOT-223 -> digikey-footprints:SOIC-14_W3.9mm; moved to F.Cu
- U6: value TL074 -> CY8C4246AZI-L445; footprint digikey-footprints:SOIC-14_W3.9mm -> digikey-footprints:LQFP-64_10x10mm; moved to F.Cu
- U7: value CY8C4246AZI-L445 -> V7805-1000; footprint digikey-footprints:LQFP-64_10x10mm -> digikey-footprints:3-SIP_Module_V7805-1000; moved to F.Cu
- moved R13 423.5 mm to (433.1, 154.6), turned to 0 degrees
- moved R14 417.3 mm to (429.9, 142.9), turned to 0 degrees
- moved RV2 414.3 mm to (418.8, 148.9), turned to 0 degrees
- moved R9 410.1 mm to (420.1, 162.5), turned to 0 degrees
- moved R5 408.7 mm to (428.8, 148.7), turned to 0 degrees
- moved R3 402.6 mm to (434.1, 142.9), turned to 0 degrees
- moved C6 399.8 mm to (434.1, 137.1), turned to 0 degrees
- moved C7 399.4 mm to (425.6, 142.9), turned to 0 degrees
- moved R8 398.0 mm to (433.1, 148.7), turned to 0 degrees
- moved C11 397.3 mm to (407.4, 162.7), turned to 0 degrees
- moved R6 396.9 mm to (424.6, 154.6), turned to 0 degrees
- moved C9 396.7 mm to (425.6, 137.1), turned to 0 degrees
- moved R2 395.5 mm to (424.6, 148.7), turned to 0 degrees
- moved R12 395.3 mm to (437.3, 148.7), turned to 0 degrees
- moved C12 392.5 mm to (429.9, 137.1)
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Connections:
- C1 pad 2: GND -> /Filters/osc1
- C13 pad 2: Net-(C13-Pad2) -> /Filters/filter_out_1
- C14 pad 1: Net-(C14-Pad1) -> Net-(C10-Pad1)
- C14 pad 2: Net-(C14-Pad2) -> /Filters/filter_out_2
- C15 pad 1: Net-(C15-Pad1) -> Net-(C11-Pad1)
- C15 pad 2: Net-(C15-Pad2) -> /Filters/filter_out_3
- C16 pad 1: Net-(C16-Pad1) -> Net-(C12-Pad1)
- C16 pad 2: Net-(C16-Pad2) -> /Filters/filter_out_4
- C17 pad 2: Net-(C17-Pad2) -> GND
- C18 pad 1: Net-(C18-Pad1) -> +15V
- C18 pad 2: Net-(C18-Pad2) -> GND
- C19 pad 1: Net-(C16-Pad1) -> +5V
- C19 pad 2: /Filters/filter_out_3 -> GND
- C2 pad 2: GND -> /Filters/osc2
- C20 pad 1: Net-(C17-Pad1) -> Net-(C20-Pad1)
- C20 pad 2: /Filters/filter_out_1 -> GND
- C21 pad 1: Net-(C18-Pad1) -> Net-(C21-Pad1)
- C21 pad 2: /Filters/filter_out_2 -> GND
- C23 pad 2: Net-(C22-Pad1) -> GND
- C24 pad 2: /Filters/osc4 -> /Envelope/lfo1
- C25 pad 2: Net-(C25-Pad2) -> /Microcontroller/envelope_pwm_1
- C26 pad 2: Net-(C26-Pad2) -> /Envelope/lfo3
- C27 pad 2: Net-(C27-Pad2) -> /Microcontroller/envelope_pwm_3
- C28 pad 1: Net-(C27-Pad1) -> Net-(C28-Pad1)
- C28 pad 2: /Filters/filter_out_4 -> /Envelope/lfo4
- C29 pad 2: GND -> /Microcontroller/envelope_pwm_4
- C3 pad 2: GND -> /Filters/osc3
- C30 pad 1: +15V -> Net-(C30-Pad1)
- C30 pad 2: GND -> /Envelope/lfo2
- C31 pad 1: +3V3 -> Net-(C31-Pad1)
- C31 pad 2: GND -> /Microcontroller/envelope_pwm_2
- C32 pad 2: /Envelope/lfo1 -> Net-(C32-Pad2)
- C33 pad 2: /Microcontroller/envelope_pwm_1 -> Net-(C33-Pad2)
- C34 pad 2: /Envelope/lfo3 -> Net-(C34-Pad2)
- C35 pad 2: /Microcontroller/envelope_pwm_3 -> Net-(C35-Pad2)
- C36 pad 2: /Envelope/lfo4 -> Net-(C32-Pad2)
- C37 pad 2: /Microcontroller/envelope_pwm_4 -> Net-(C33-Pad2)
- C38 pad 2: /Envelope/lfo2 -> Net-(C34-Pad2)
- C39 pad 2: /Microcontroller/envelope_pwm_2 -> Net-(C35-Pad2)
- C4 pad 2: Net-(C1-Pad1) -> /Filters/osc4
- C44 pad 2: Net-(C40-Pad2) -> /Envelope/env_out_1
- C45 pad 2: Net-(C41-Pad2) -> /Envelope/env_out_2
- C46 pad 2: Net-(C42-Pad2) -> /Envelope/env_out_3
- C47 pad 2: Net-(C43-Pad2) -> /Envelope/env_out_4
- C49 pad 1: Net-(C49-Pad1) -> +5V
- C49 pad 2: Net-(C49-Pad2) -> GND
- C5 pad 2: /Filters/osc3 -> GND
- C50 pad 1: Net-(C50-Pad1) -> +5V
- C50 pad 2: Net-(C50-Pad2) -> GND
- C51 pad 2: Net-(C51-Pad2) -> GND
- C52 pad 1: Net-(C52-Pad1) -> Net-(C48-Pad1)
- C52 pad 2: /Envelope/env_out_1 -> /Mixer and Effects/delay_in
- C53 pad 2: /Envelope/env_out_2 -> GND
- C54 pad 2: /Envelope/env_out_3 -> GND
- C55 pad 2: /Envelope/env_out_4 -> Net-(C55-Pad2)
- C57 pad 1: Net-(C56-Pad1) -> Net-(C57-Pad1)
- C59 pad 1: Net-(C58-Pad2) -> Net-(C59-Pad1)
- C59 pad 2: /LFO Modulation and Routing/lfo_tri -> GND
- C6 pad 2: Net-(C2-Pad1) -> GND
- C60 pad 2: /LFO Modulation and Routing/main_lfo -> GND
- C61 pad 2: /LFO Modulation and Routing/main_lfo -> Net-(C61-Pad2)
- C63 pad 1: Net-(C63-Pad1) -> Net-(C59-Pad1)
- C64 pad 1: Net-(C62-Pad2) -> Net-(C64-Pad1)
- C64 pad 2: Net-(C64-Pad2) -> GND
- C65 pad 1: Net-(C63-Pad2) -> Net-(C65-Pad1)
- C65 pad 2: Net-(C65-Pad2) -> /Mixer and Effects/delay_in
- C66 pad 1: Net-(C66-Pad1) -> Net-(C64-Pad1)
- C66 pad 2: /LFO Modulation and Routing/main_lfo -> Net-(C66-Pad2)
- C67 pad 2: /LFO Modulation and Routing/main_lfo -> Net-(C67-Pad2)
- C69 pad 1: Net-(C69-Pad1) -> Net-(C68-Pad1)
- C7 pad 2: /Filters/osc1 -> GND
- C70 pad 1: Net-(C68-Pad2) -> Net-(C70-Pad1)
- C71 pad 1: Net-(C69-Pad2) -> Net-(C71-Pad1)
- C71 pad 2: Net-(C71-Pad2) -> /LFO Modulation and Routing/lfo_square
- C72 pad 2: GNDD -> Net-(C72-Pad2)
- C73 pad 1: Net-(C73-Pad1) -> Net-(C72-Pad2)
- C73 pad 2: GNDD -> /LFO Modulation and Routing/lfo_tri
- C74 pad 1: +3V3 -> Net-(C74-Pad1)
- C74 pad 2: GNDD -> Net-(C74-Pad2)
- C75 pad 1: +3V3 -> Net-(C75-Pad1)
- C75 pad 2: GNDD -> Net-(C75-Pad2)
- C76 pad 1: +3V3 -> Net-(C76-Pad1)
- C76 pad 2: GNDD -> Net-(C76-Pad2)
- C77 pad 1: +3V3 -> Net-(C77-Pad1)
- C77 pad 2: GNDD -> Net-(C77-Pad2)
- C78 pad 1: +3V3 -> +5V
- C79 pad 1: +3V3 -> +5V
- C8 pad 2: Net-(C3-Pad1) -> GND
- C80 pad 1: +3V3 -> +5V
- C81 pad 1: +3V3 -> +5V
- C9 pad 1: Net-(C9-Pad1) -> Net-(C13-Pad1)
- C9 pad 2: /Filters/osc2 -> Net-(C9-Pad2)
- D2 pad 1: /LFO Modulation and Routing/lfo_square -> Net-(C71-Pad1)
- J2 pad 1: Net-(C57-Pad2) -> Net-(C69-Pad2)
- J3 pad 1: +3V3 -> +5V
- Q1 pad 1: Net-(C40-Pad2) -> Net-(C20-Pad1)
- Q1 pad 2: GND -> /Envelope/lfo_bias_1
- Q1 pad 3: Net-(Q1-Pad3) -> +15V
- Q2 pad 1: Net-(C41-Pad2) -> Net-(C21-Pad1)
- Q2 pad 2: GND -> /Envelope/lfo_bias_2
- Q2 pad 3: Net-(Q2-Pad3) -> +15V
- Q3 pad 1: Net-(C42-Pad2) -> Net-(C22-Pad1)
- Q3 pad 2: GND -> /Envelope/lfo_bias_3
- Q3 pad 3: Net-(Q3-Pad3) -> +15V
- Q4 pad 1: Net-(C43-Pad2) -> Net-(C23-Pad1)
- Q4 pad 2: GND -> /Envelope/lfo_bias_4
- Q4 pad 3: Net-(Q4-Pad3) -> +15V
- Q5 pad 1: Net-(Q5-Pad1) -> Net-(C32-Pad2)
- Q5 pad 2: Net-(C60-Pad1) -> GND
- Q5 pad 3: Net-(C62-Pad1) -> Net-(Q5-Pad3)
- Q6 pad 1: Net-(Q6-Pad1) -> Net-(C33-Pad2)
- Q6 pad 2: Net-(C61-Pad1) -> GND
- Q6 pad 3: Net-(C63-Pad1) -> Net-(Q6-Pad3)
- Q7 pad 1: Net-(Q7-Pad1) -> Net-(C34-Pad2)
- Q7 pad 2: Net-(C66-Pad1) -> GND
- Q7 pad 3: Net-(C68-Pad1) -> Net-(Q7-Pad3)
- Q8 pad 1: Net-(Q8-Pad1) -> Net-(C35-Pad2)
- Q8 pad 2: Net-(C67-Pad1) -> GND
- Q8 pad 3: Net-(C69-Pad1) -> Net-(Q8-Pad3)
- R1 pad 1: Net-(C1-Pad1) -> Net-(R1-Pad1)
- R1 pad 2: /Filters/osc3 -> Net-(C1-Pad1)
- R10 pad 1: Net-(C16-Pad2) -> VREF
- R10 pad 2: Net-(C13-Pad2) -> Net-(C6-Pad1)
- R100 pad 1: +3V3 -> /Microcontroller/osc3_quant
- R100 pad 2: Net-(R100-Pad2) -> +5V
- R101 pad 1: +3V3 -> /Microcontroller/osc2_quant
- R101 pad 2: Net-(R101-Pad2) -> +5V
- R102 pad 1: +3V3 -> /Microcontroller/osc1_quant
- R102 pad 2: Net-(R102-Pad2) -> +5V
- R103 pad 1: +3V3 -> +5V
- R104 pad 1: +3V3 -> +5V
- R105 pad 1: +3V3 -> +5V
- R106 pad 1: +3V3 -> +5V
- R106 pad 2: /Microcontroller/XRES -> Net-(R106-Pad2)
- R107 pad 1: GND -> +5V
- R107 pad 2: GNDD -> Net-(R107-Pad2)
- R11 pad 1: Net-(C16-Pad2) -> VREF
- R11 pad 2: Net-(C10-Pad2) -> Net-(C7-Pad1)
- R12 pad 1: Net-(C17-Pad2) -> VREF
- R12 pad 2: Net-(C14-Pad2) -> Net-(C8-Pad1)
- R13 pad 1: Net-(C17-Pad2) -> /Filters/filter_out_1
- R13 pad 2: Net-(C11-Pad2) -> GND
- R14 pad 1: Net-(C18-Pad2) -> /Filters/filter_out_2
- R14 pad 2: Net-(C15-Pad2) -> GND
- R15 pad 1: Net-(C18-Pad2) -> /Filters/filter_out_3
- R15 pad 2: Net-(C12-Pad2) -> GND
- R16 pad 1: Net-(R16-Pad1) -> /Filters/filter_out_4
- R16 pad 2: VREF -> GND
- R17 pad 1: Net-(R17-Pad1) -> +15V
- R17 pad 2: VREF -> Net-(C17-Pad1)
- R18 pad 1: Net-(R18-Pad1) -> Net-(C17-Pad1)
- R18 pad 2: VREF -> GND
- R19 pad 1: Net-(C16-Pad1) -> /Envelope/lfo_bias_1
- R19 pad 2: Net-(C16-Pad2) -> GND
- R2 pad 1: Net-(C2-Pad1) -> Net-(R2-Pad1)
- R2 pad 2: /Filters/osc1 -> Net-(C2-Pad1)
- R20 pad 1: Net-(C17-Pad1) -> /Envelope/lfo_bias_2
- R20 pad 2: Net-(C17-Pad2) -> GND
- R21 pad 1: Net-(C18-Pad1) -> /Envelope/lfo_bias_3
- R21 pad 2: Net-(C18-Pad2) -> GND
- R22 pad 1: /Filters/filter_out_3 -> /Envelope/lfo_bias_4
- R23 pad 1: /Filters/filter_out_1 -> /Envelope/lfo_bias_3
- R23 pad 2: GND -> Net-(C26-Pad1)
- R24 pad 1: /Filters/filter_out_2 -> /Envelope/lfo_bias_4
- R24 pad 2: GND -> Net-(C28-Pad1)
- R25 pad 1: Net-(C22-Pad1) -> /Envelope/lfo_bias_1
- R25 pad 2: /Filters/osc4 -> Net-(C24-Pad1)
- R26 pad 1: VREF -> /Envelope/lfo_bias_2
- R26 pad 2: Net-(C24-Pad1) -> Net-(C30-Pad1)
- R27 pad 1: VREF -> Net-(R27-Pad1)
- R27 pad 2: Net-(C23-Pad1) -> Net-(C24-Pad1)
- R28 pad 1: Net-(C27-Pad2) -> Net-(R27-Pad1)
- R28 pad 2: Net-(C26-Pad2) -> Net-(C25-Pad1)
- R29 pad 1: Net-(C27-Pad2) -> Net-(R29-Pad1)
- R29 pad 2: Net-(C25-Pad2) -> Net-(C30-Pad1)
- R3 pad 1: Net-(C3-Pad1) -> Net-(R3-Pad1)
- R3 pad 2: /Filters/osc2 -> Net-(C3-Pad1)
- R30 pad 1: Net-(R30-Pad1) -> Net-(R29-Pad1)
- R30 pad 2: VREF -> Net-(C31-Pad1)
- R31 pad 1: Net-(C27-Pad1) -> Net-(R31-Pad1)
- R31 pad 2: Net-(C27-Pad2) -> Net-(C26-Pad1)
- R32 pad 1: /Filters/filter_out_4 -> Net-(R31-Pad1)
- R32 pad 2: GND -> Net-(C27-Pad1)
- R33 pad 1: +15V -> Net-(R33-Pad1)
- R33 pad 2: Net-(C29-Pad1) -> Net-(C28-Pad1)
- R34 pad 1: Net-(C29-Pad1) -> Net-(R33-Pad1)
- R34 pad 2: GND -> Net-(C29-Pad1)
- R35 pad 1: /Envelope/lfo_bias -> Net-(C32-Pad2)
- R35 pad 2: +15V -> /Filters/filter_out_1
- R36 pad 1: GND -> Net-(C33-Pad2)
- R36 pad 2: /Envelope/lfo_bias -> /Filters/filter_out_2
- R37 pad 1: /Envelope/lfo_bias -> Net-(C34-Pad2)
- R37 pad 2: Net-(C34-Pad1) -> /Filters/filter_out_3
- R38 pad 1: /Envelope/lfo_bias -> Net-(C35-Pad2)
- R38 pad 2: Net-(C36-Pad1) -> /Filters/filter_out_4
- R39 pad 1: /Envelope/lfo_bias -> Net-(Q5-Pad3)
- R39 pad 2: Net-(C32-Pad1) -> Net-(R27-Pad1)
- R4 pad 1: VREF -> Net-(R4-Pad1)
- R4 pad 2: Net-(C5-Pad1) -> Net-(C4-Pad1)
- R40 pad 1: /Envelope/lfo_bias -> Net-(Q6-Pad3)
- R40 pad 2: Net-(C38-Pad1) -> Net-(R29-Pad1)
- R41 pad 1: Net-(R41-Pad1) -> Net-(Q7-Pad3)
- R41 pad 2: Net-(C32-Pad1) -> Net-(R31-Pad1)
- R42 pad 1: Net-(R41-Pad1) -> Net-(Q8-Pad3)
- R42 pad 2: Net-(C33-Pad1) -> Net-(R33-Pad1)
- R43 pad 1: Net-(R43-Pad1) -> Net-(Q5-Pad3)
- R43 pad 2: Net-(C38-Pad1) -> Net-(C32-Pad1)
- R44 pad 1: Net-(R43-Pad1) -> Net-(Q6-Pad3)
- R44 pad 2: Net-(C39-Pad1) -> Net-(C33-Pad1)
- R45 pad 1: Net-(R45-Pad1) -> Net-(Q7-Pad3)
- R46 pad 1: Net-(R45-Pad1) -> Net-(Q8-Pad3)
- R47 pad 1: Net-(R47-Pad1) -> Net-(C37-Pad1)
- R47 pad 2: Net-(C36-Pad1) -> VREF
- R48 pad 1: Net-(R47-Pad1) -> Net-(C38-Pad1)
- R48 pad 2: Net-(C37-Pad1) -> VREF
- R49 pad 1: Net-(C40-Pad2) -> Net-(C39-Pad1)
- R49 pad 2: /Filters/filter_out_1 -> VREF
- R5 pad 1: VREF -> Net-(C5-Pad1)
- R5 pad 2: Net-(C7-Pad1) -> Net-(R5-Pad2)
- R50 pad 1: Net-(C41-Pad2) -> Net-(C36-Pad1)
- R50 pad 2: /Filters/filter_out_2 -> VREF
- R51 pad 1: Net-(C42-Pad2) -> Net-(C48-Pad2)
- R51 pad 2: /Filters/filter_out_3 -> Net-(C44-Pad1)
- R52 pad 1: Net-(C43-Pad2) -> Net-(C48-Pad2)
- R52 pad 2: /Filters/filter_out_4 -> Net-(C45-Pad1)
- R53 pad 1: Net-(Q1-Pad3) -> Net-(C48-Pad2)
- R53 pad 2: Net-(R41-Pad1) -> Net-(C46-Pad1)
- R54 pad 1: Net-(Q2-Pad3) -> Net-(C48-Pad2)
- R54 pad 2: Net-(R43-Pad1) -> Net-(C47-Pad1)
- R55 pad 1: Net-(Q3-Pad3) -> Net-(R55-Pad1)
- R55 pad 2: Net-(R45-Pad1) -> VREF
- R56 pad 1: Net-(Q4-Pad3) -> Net-(C48-Pad1)
- R56 pad 2: Net-(R47-Pad1) -> Net-(C48-Pad2)
- R57 pad 1: Net-(Q1-Pad3) -> Net-(R57-Pad1)
- R57 pad 2: Net-(C40-Pad1) -> Net-(R57-Pad2)
- R58 pad 1: Net-(Q2-Pad3) -> GND
- R58 pad 2: Net-(C41-Pad1) -> /Mixer and Effects/delay_in
- R59 pad 1: Net-(Q3-Pad3) -> Net-(C61-Pad2)
- R59 pad 2: Net-(C42-Pad1) -> /Mixer and Effects/delay_in
- R6 pad 1: VREF -> Net-(C6-Pad1)
- R6 pad 2: Net-(C9-Pad1) -> Net-(R6-Pad2)
- R60 pad 1: Net-(Q4-Pad3) -> Net-(C62-Pad2)
- R60 pad 2: Net-(C43-Pad1) -> /Mixer and Effects/delay_out
- R61 pad 1: Net-(C45-Pad1) -> Net-(R61-Pad1)
- R62 pad 1: Net-(C46-Pad1) -> Net-(R62-Pad1)
- R63 pad 1: Net-(C47-Pad1) -> Net-(C59-Pad1)
- R63 pad 2: VREF -> Net-(C55-Pad1)
- R64 pad 1: Net-(C44-Pad1) -> Net-(C59-Pad1)
- R64 pad 2: VREF -> Net-(C55-Pad2)
- R65 pad 1: Net-(C56-Pad2) -> Net-(C60-Pad1)
- R65 pad 2: Net-(C52-Pad1) -> Net-(C56-Pad1)
- R66 pad 1: Net-(C56-Pad2) -> Net-(C60-Pad1)
- R66 pad 2: Net-(C53-Pad1) -> Net-(C56-Pad2)
- R67 pad 1: Net-(C56-Pad2) -> Net-(C60-Pad1)
- R67 pad 2: Net-(C54-Pad1) -> Net-(C57-Pad1)
- R68 pad 1: Net-(C56-Pad2) -> Net-(C61-Pad1)
- R68 pad 2: Net-(C55-Pad1) -> Net-(C61-Pad2)
- R69 pad 1: Net-(R69-Pad1) -> Net-(C62-Pad1)
- R69 pad 2: VREF -> Net-(C62-Pad2)
- R7 pad 1: VREF -> Net-(C7-Pad1)
- R7 pad 2: Net-(C4-Pad1) -> Net-(R7-Pad2)
- R70 pad 1: Net-(C56-Pad1) -> Net-(C65-Pad1)
- R70 pad 2: Net-(C56-Pad2) -> Net-(C59-Pad1)
- R71 pad 1: GND -> Net-(C64-Pad1)
- R71 pad 2: Net-(C57-Pad2) -> Net-(C56-Pad1)
- R72 pad 1: +15V -> GND
- R72 pad 2: /LFO Modulation and Routing/bias -> /Mixer and Effects/delay_in
- R73 pad 1: /LFO Modulation and Routing/bias -> Net-(C63-Pad2)
- R73 pad 2: GND -> Net-(R73-Pad2)
- R74 pad 1: Net-(R74-Pad1) -> Net-(C68-Pad2)
- R74 pad 2: VREF -> Net-(C61-Pad1)
- R75 pad 1: Net-(R75-Pad1) -> Net-(C68-Pad2)
- R75 pad 2: Net-(R75-Pad2) -> Net-(C62-Pad1)
- R76 pad 2: Net-(R75-Pad1) -> VREF
- R77 pad 1: Net-(C58-Pad2) -> Net-(C55-Pad2)
- R77 pad 2: Net-(R75-Pad2) -> Net-(C67-Pad1)
- R78 pad 1: /LFO Modulation and Routing/lfo_square -> Net-(C68-Pad1)
- R78 pad 2: Net-(R75-Pad1) -> Net-(C68-Pad2)
- R79 pad 1: Net-(R79-Pad1) -> GND
- R79 pad 2: VREF -> Net-(C69-Pad2)
- R8 pad 1: VREF -> Net-(C8-Pad1)
- R8 pad 2: Net-(C6-Pad1) -> Net-(R8-Pad2)
- R80 pad 1: GND -> Net-(R80-Pad1)
- R80 pad 2: /LFO Modulation and Routing/lfo_tri -> VREF
- R81 pad 1: /LFO Modulation and Routing/bias -> Net-(C70-Pad1)
- R81 pad 2: Net-(C60-Pad1) -> Net-(R81-Pad2)
- R82 pad 1: /LFO Modulation and Routing/bias -> Net-(R82-Pad1)
- R82 pad 2: Net-(C61-Pad1) -> Net-(C70-Pad1)
- R83 pad 1: +15V -> Net-(C72-Pad2)
- R83 pad 2: Net-(C62-Pad1) -> Net-(R81-Pad2)
- R84 pad 1: Net-(Q5-Pad1) -> Net-(C71-Pad1)
- R84 pad 2: GND -> Net-(C70-Pad2)
- R85 pad 1: +15V -> Net-(C71-Pad1)
- R85 pad 2: Net-(C63-Pad1) -> GND
- R86 pad 1: Net-(Q6-Pad1) -> Net-(R86-Pad1)
- R86 pad 2: GND -> VREF
- R87 pad 1: /LFO Modulation and Routing/bias -> GND
- R87 pad 2: Net-(C66-Pad1) -> /LFO Modulation and Routing/lfo_tri
- R88 pad 1: /LFO Modulation and Routing/bias -> Net-(R88-Pad1)
- R88 pad 2: Net-(C67-Pad1) -> VREF
- R89 pad 1: +15V -> /LFO Modulation and Routing/main_lfo
- R89 pad 2: Net-(C68-Pad1) -> VREF
- R9 pad 2: Net-(C8-Pad1) -> Net-(C5-Pad1)
- R90 pad 1: Net-(Q7-Pad1) -> /LFO Modulation and Routing/main_lfo
- R90 pad 2: GND -> VREF
- R91 pad 1: +15V -> /LFO Modulation and Routing/main_lfo
- R91 pad 2: Net-(C69-Pad1) -> VREF
- R92 pad 1: Net-(Q8-Pad1) -> GND
- R92 pad 2: GND -> GNDD
- R93 pad 1: Net-(C73-Pad1) -> Net-(C87-Pad1)
- R93 pad 2: Net-(C72-Pad1) -> Net-(C82-Pad1)
- R94 pad 1: +3V3 -> +5V
- R94 pad 2: Net-(R94-Pad2) -> /Microcontroller/XRES
- R95 pad 1: +3V3 -> /Microcontroller/osc4_repeat
- R95 pad 2: Net-(R95-Pad2) -> +5V
- R96 pad 1: +3V3 -> /Microcontroller/osc3_repeat
- R96 pad 2: Net-(R96-Pad2) -> +5V
- R97 pad 1: +3V3 -> /Microcontroller/osc2_repeat
- R97 pad 2: Net-(R97-Pad2) -> +5V
- R98 pad 1: +3V3 -> /Microcontroller/osc1_repeat
- R98 pad 2: Net-(R98-Pad2) -> +5V
- R99 pad 1: +3V3 -> /Microcontroller/osc4_quant
- R99 pad 2: Net-(R99-Pad2) -> +5V
- RV1 pad 1: Net-(C13-Pad2) -> Net-(R1-Pad1)
- RV1 pad 2: GND -> Net-(R1-Pad1)
- RV1 pad 3: Net-(C10-Pad2) -> Net-(C9-Pad2)
- RV10 pad 1: Net-(C62-Pad2) -> Net-(C41-Pad2)
- RV10 pad 2: Net-(C62-Pad2) -> /Envelope/env_out_2
- RV10 pad 3: Net-(Q5-Pad1) -> GND
- RV11 pad 1: Net-(C63-Pad2) -> Net-(C42-Pad2)
- RV11 pad 2: Net-(C63-Pad2) -> /Envelope/env_out_3
- RV11 pad 3: Net-(Q6-Pad1) -> GND
- RV12 pad 1: Net-(C64-Pad2) -> Net-(C43-Pad2)
- RV12 pad 2: /Envelope/lfo3 -> /Envelope/env_out_4
- RV13 pad 1: Net-(C65-Pad2) -> Net-(R57-Pad2)
- RV13 pad 2: /Envelope/lfo1 -> Net-(R57-Pad2)
- RV14 pad 1: Net-(C68-Pad2) -> /Mixer and Effects/delay_in
- RV14 pad 2: Net-(C68-Pad2) -> GND
- RV14 pad 3: Net-(Q7-Pad1) -> /Mixer and Effects/delay_out
- RV15 pad 1: Net-(C69-Pad2) -> Net-(C66-Pad2)
- RV15 pad 2: Net-(C69-Pad2) -> Net-(R73-Pad2)
- RV15 pad 3: Net-(Q8-Pad1) -> GND
- RV16 pad 1: Net-(C70-Pad2) -> Net-(C67-Pad2)
- RV16 pad 2: /Envelope/lfo2 -> /Mixer and Effects/delay_out
- RV17 pad 1: Net-(C71-Pad2) -> Net-(C72-Pad1)
- RV17 pad 2: /Envelope/lfo4 -> Net-(R82-Pad1)
- RV17 pad 3: GND -> Net-(R82-Pad1)
- RV18 pad 1: Net-(R94-Pad2) -> Net-(C74-Pad2)
- RV18 pad 2: /Microcontroller/osc1_freq_wiper -> /Envelope/lfo3
- RV19 pad 1: Net-(R95-Pad2) -> Net-(C75-Pad2)
- RV19 pad 2: /Microcontroller/osc2_freq_wiper -> /Envelope/lfo1
- RV2 pad 1: Net-(C14-Pad2) -> Net-(R2-Pad1)
- RV2 pad 2: GND -> Net-(R2-Pad1)
- RV2 pad 3: Net-(C11-Pad2) -> Net-(C10-Pad2)
- RV20 pad 1: Net-(R96-Pad2) -> Net-(C76-Pad2)
- RV20 pad 2: /Microcontroller/osc3_freq_wiper -> /Envelope/lfo2
- RV21 pad 1: Net-(R97-Pad2) -> Net-(C77-Pad2)
- RV21 pad 2: /Microcontroller/osc4_freq_wiper -> /Envelope/lfo4
- RV22 pad 1: Net-(R98-Pad2) -> Net-(R103-Pad2)
- RV22 pad 2: /Microcontroller/osc1_pwm_wiper -> /Microcontroller/osc1_freq_wiper
- RV23 pad 1: Net-(R99-Pad2) -> Net-(R104-Pad2)
- RV23 pad 2: /Microcontroller/osc2_pwm_wiper -> /Microcontroller/osc2_freq_wiper
- RV24 pad 1: Net-(R100-Pad2) -> Net-(R105-Pad2)
- RV24 pad 2: /Microcontroller/osc3_pwm_wiper -> /Microcontroller/osc3_freq_wiper
- RV25 pad 1: Net-(R101-Pad2) -> Net-(R106-Pad2)
- RV25 pad 2: /Microcontroller/osc4_pwm_wiper -> /Microcontroller/osc4_freq_wiper
- RV26 pad 1: Net-(R102-Pad2) -> Net-(R107-Pad2)
- RV26 pad 2: /Microcontroller/osc1_speed -> /Microcontroller/osc1_pwm_wiper
- RV27 pad 1: Net-(R103-Pad2) -> Net-(R108-Pad2)
- RV27 pad 2: /Microcontroller/osc2_speed -> /Microcontroller/osc2_pwm_wiper
- RV28 pad 1: Net-(R104-Pad2) -> Net-(R109-Pad2)
- RV28 pad 2: /Microcontroller/osc3_speed -> /Microcontroller/osc3_pwm_wiper
- RV29 pad 1: Net-(R105-Pad2) -> Net-(R110-Pad2)
- RV29 pad 2: /Microcontroller/osc4_speed -> /Microcontroller/osc4_pwm_wiper
- RV3 pad 1: Net-(C15-Pad2) -> Net-(R3-Pad1)
- RV3 pad 2: GND -> Net-(R3-Pad1)
- RV3 pad 3: Net-(C12-Pad2) -> Net-(C11-Pad2)
- RV4 pad 1: Net-(C26-Pad2) -> Net-(R4-Pad1)
- RV4 pad 2: GND -> Net-(R4-Pad1)
- RV4 pad 3: Net-(C25-Pad2) -> Net-(C12-Pad2)
- RV5 pad 1: Net-(C48-Pad2) -> +15V
- RV5 pad 2: /Envelope/env_out_1 -> Net-(C20-Pad1)
- RV6 pad 1: Net-(C49-Pad2) -> +15V
- RV6 pad 2: /Envelope/env_out_2 -> Net-(C21-Pad1)
- RV7 pad 1: Net-(C50-Pad2) -> +15V
- RV7 pad 2: /Envelope/env_out_3 -> Net-(C22-Pad1)
- RV8 pad 1: Net-(C51-Pad2) -> +15V
- RV8 pad 2: /Envelope/env_out_4 -> Net-(C23-Pad1)
- RV9 pad 1: Net-(C58-Pad1) -> Net-(C40-Pad2)
- RV9 pad 2: Net-(C58-Pad1) -> /Envelope/env_out_1
- RV9 pad 3: Net-(R76-Pad1) -> GND
- U1 pad 10: Net-(C23-Pad1) -> Net-(C7-Pad1)
- U1 pad 11: +15V -> GND
- U1 pad 12: Net-(C24-Pad1) -> Net-(C8-Pad1)
- U1 pad 13: Net-(C25-Pad1) -> Net-(C12-Pad1)
- U1 pad 14: Net-(C25-Pad1) -> Net-(C12-Pad1)
- U1 pad 2: Net-(C4-Pad1) -> Net-(C13-Pad1)
- U1 pad 3: Net-(C13-Pad1) -> Net-(C5-Pad1)
- U1 pad 4: GND -> +15V
- U1 pad 5: Net-(C5-Pad1) -> Net-(C6-Pad1)
- U1 pad 8: Net-(C26-Pad1) -> Net-(C11-Pad1)
- U1 pad 9: Net-(C26-Pad1) -> Net-(C11-Pad1)
- U2 pad 1: Net-(C14-Pad1) -> Net-(C40-Pad1)
- U2 pad 10: Net-(C8-Pad1) -> Net-(C38-Pad1)
- U2 pad 12: Net-(C9-Pad1) -> Net-(C39-Pad1)
- U2 pad 13: Net-(C12-Pad1) -> Net-(C43-Pad1)
- U2 pad 14: Net-(C12-Pad1) -> Net-(C43-Pad1)
- U2 pad 2: Net-(C14-Pad1) -> Net-(C40-Pad1)
- U2 pad 3: Net-(C6-Pad1) -> Net-(C36-Pad1)
- U2 pad 5: Net-(C7-Pad1) -> Net-(C37-Pad1)
- U2 pad 6: Net-(C11-Pad1) -> Net-(C41-Pad1)
- U2 pad 7: Net-(C11-Pad1) -> Net-(C41-Pad1)
- U2 pad 8: Net-(C15-Pad1) -> Net-(C42-Pad1)
- U2 pad 9: Net-(C15-Pad1) -> Net-(C42-Pad1)
- U3 pad 1: Net-(C17-Pad1) -> Net-(C48-Pad1)
- U3 pad 10: Net-(R16-Pad1) -> Net-(R62-Pad1)
- U3 pad 12: Net-(R30-Pad1) -> Net-(R76-Pad1)
- U3 pad 13: Net-(C27-Pad2) -> Net-(C68-Pad2)
- U3 pad 14: Net-(C27-Pad1) -> Net-(C68-Pad1)
- U3 pad 2: Net-(C17-Pad2) -> Net-(C48-Pad2)
- U3 pad 3: Net-(R17-Pad1) -> Net-(R55-Pad1)
- U3 pad 5: Net-(R18-Pad1) -> Net-(R61-Pad1)
- U3 pad 6: Net-(C18-Pad2) -> Net-(C61-Pad2)
- U3 pad 7: Net-(C18-Pad1) -> Net-(C61-Pad1)
- U3 pad 8: Net-(C16-Pad1) -> Net-(C62-Pad1)
- U3 pad 9: Net-(C16-Pad2) -> Net-(C62-Pad2)
- U4 pad 1: Net-(R75-Pad1) -> Net-(C70-Pad1)
- U4 pad 10: Net-(R69-Pad1) -> Net-(C17-Pad1)
- U4 pad 12: Net-(C29-Pad1) -> (no net)
- U4 pad 13: VREF -> (no net)
- U4 pad 14: VREF -> (no net)
- U4 pad 2: Net-(R74-Pad1) -> Net-(R80-Pad1)
- U4 pad 3: Net-(R75-Pad2) -> Net-(R81-Pad2)
- U4 pad 5: Net-(R79-Pad1) -> Net-(R86-Pad1)
- U4 pad 6: Net-(C58-Pad1) -> Net-(C72-Pad1)
- U4 pad 7: Net-(C58-Pad2) -> Net-(C72-Pad2)
- U4 pad 8: Net-(C56-Pad1) -> VREF
- U4 pad 9: Net-(C56-Pad2) -> VREF
- U5 pad 1: GND -> Net-(C75-Pad1)
- U5 pad 2: +3V3 -> Net-(C75-Pad1)
- U5 pad 3: +15V -> /LFO Modulation and Routing/main_lfo
- U5 pad 4: +3V3 -> +15V
- U6 pad 1: Net-(C48-Pad1) -> /Microcontroller/osc1_speed
- U6 pad 10: Net-(C46-Pad1) -> GNDD
- U6 pad 11: GND -> +5V
- U6 pad 12: Net-(C47-Pad1) -> Net-(U6-Pad12)
- U6 pad 13: Net-(C51-Pad1) -> Net-(U6-Pad13)
- U6 pad 14: Net-(C51-Pad1) -> /Filters/osc1
- U6 pad 2: Net-(C48-Pad1) -> /Microcontroller/osc1_freq_wiper
- U6 pad 3: Net-(C44-Pad1) -> /Microcontroller/osc1_pwm_wiper
- U6 pad 4: +15V -> /Microcontroller/osc2_freq_wiper
- U6 pad 5: Net-(C45-Pad1) -> /Microcontroller/osc2_pwm_wiper
- U6 pad 6: Net-(C49-Pad1) -> /Microcontroller/osc3_freq_wiper
- U6 pad 7: Net-(C49-Pad1) -> /Microcontroller/osc3_pwm_wiper
- U6 pad 8: Net-(C50-Pad1) -> /Microcontroller/osc4_freq_wiper
- U6 pad 9: Net-(C50-Pad1) -> /Microcontroller/osc4_pwm_wiper
- U7 pad 1: /Microcontroller/osc1_speed -> +15V
- U7 pad 2: /Microcontroller/osc1_freq_wiper -> GND
- U7 pad 3: /Microcontroller/osc1_pwm_wiper -> +5V
- Y1 pad 1: Net-(C72-Pad1) -> Net-(C82-Pad1)
- Y1 pad 2: Net-(C73-Pad1) -> Net-(C87-Pad1)
Routing:
- net +3V3: track 644.9 -> 0.00 mm, vias 7 -> 0
- net +15V: track 477.5 -> 0.00 mm, vias 12 -> 0
- net GND: track 366.2 -> 0.00 mm, vias 27 -> 0
- net /Envelope/lfo_bias: track 250.1 -> 0.00 mm, vias 4 -> 0
- net /LFO Modulation and Routing/bias: track 247.9 -> 0.00 mm, vias 7 -> 0
- net GNDD: track 233.1 -> 0.00 mm, vias 4 -> 0
- net /Envelope/lfo1: track 198.0 -> 0.00 mm, vias 1 -> 0
- net VREF: track 195.3 -> 0.00 mm, vias 25 -> 0
- net /LFO Modulation and Routing/main_lfo: track 185.8 -> 0.00 mm, vias 5 -> 0
- net /Filters/osc4: track 181.9 -> 0.00 mm, vias 2 -> 0
- net /Microcontroller/osc4_freq_wiper: track 167.3 -> 0.00 mm, vias 1 -> 0
- net /Microcontroller/osc4_pwm_wiper: track 166.4 -> 0.00 mm, vias 1 -> 0
- net /Filters/filter_out_4: track 158.9 -> 0.00 mm, vias 2 -> 0
- net /Filters/osc3: track 150.1 -> 0.00 mm, vias 2 -> 0
- net /Microcontroller/osc4_speed: track 148.9 -> 0.00 mm, vias 1 -> 0
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- removed copper zone on B.Cu, net GND
- removed copper zone on F.Cu, net GND
- removed copper zone on In2.Cu, net GND
- removed copper zone on In1.Cu, net VREF
Other:
- board outline removed
- copper layers 4 -> 2
- net class PWR removed
- rule pad_to_mask_clearance: 0.2 -> 0
