File: Hardware/synth_psoc.sch (KiCad schematic (older format))
At the start: 0 parts

Commit message: add analog LFO to schematic
Changed lines of the file:
@@
 F4 "osc3" I L 7500 3250 60
 F5 "osc4" I L 7500 3350 60
-F6 "mix_out" O R 8100 3500 60
 $EndSheet
 $Sheet

Commit message: simulate bias voltage buffer. Previous op amp approach couldn't go close enough to the rails.
Changed lines of the file:
@@
 S 7500 3000 600  800
 U 5C357081
-F0 "Mixer and output connectors" 60
+F0 "Mixer and Effects" 60
 F1 "mixer.sch" 60
 F2 "osc1" I L 7500 3050 60
