File: Hardware/vcf.sch (KiCad schematic (older format))
At the start: 40 parts, among them U2 TL074

Commit message: begin PCB v2 layout. fix ref designators, associate footprints on new components, create new PCB file, import components.
Parts:
- gave numbers to parts that had none: 34
- renumbered C6 to C1, C2 to C5, R8 to R9, U2 to U1
Connections:
- net at C10.1, C14.1: now also U1.6 (-), U1.7; no longer U1.1, U1.2 (-)
- net at C6.1, R10.2, R6.1: now also U1.5 (+); no longer U1.3 (+)
- net at C11.1, C15.1: now also U1.8, U1.9 (-); no longer U1.1, U1.2 (-)
- net at C7.1, R11.2, R7.1: now also U1.10 (+); no longer U1.3 (+)
- net at C12.1, C16.1: now also U1.13 (-), U1.14; no longer U1.1, U1.2 (-)
- net at C8.1, R12.2, R8.1: now also U1.12 (+); no longer U1.3 (+)
