File: Hardware/Synth Engine/mcu.sch (KiCad schematic (older format))
At the start: 74 parts, among them J3 SWD_programming, J4 Capsense_0, J5 Capsense_1, J6 Capsense_2, J7 Capsense_3, SW10 SW_SPST, SW11 SW_SPST, SW12 SW_SPST, SW13 SW_SPST, SW2 SW_SPST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

Commit message: add separate Kicad project for control board. There will now be a separate board for all potentiometers and switches with no other components. Also add connectors between boards.
Parts:
- C78, C79, C83, C86, C88: footprint Capacitors_SMD:C_0805 -> Capacitors_SMD:CP_Elec_4x4.5
- C80, C81, C84, C85: footprint Capacitors_SMD:C_0805 -> digikey-footprints:0805
- C89: footprint (none) -> digikey-footprints:0805
- C90, C91, C92, C93: footprint (none) -> Capacitors_SMD:CP_Elec_5x5.7
- SW10, SW11, SW12, SW13, SW2, SW3, SW4, SW5, SW6, SW7, SW8, SW9: footprint (none) -> SparkFun-Electromechanical:SWITCH-SPDT
