File: Hardware/Synth Engine/mixer.sch (KiCad schematic (older format))
At the start: 62 parts, among them J2 Audio-Jack-2_Switch, U3 TL074, U8 PT2399

Commit message: add separate Kicad project for control board. There will now be a separate board for all potentiometers and switches with no other components. Also add connectors between boards.
Parts:
- R57, R63, R64, R65, R66, R67, R70, R71, R72, R73, R77: footprint (none) -> digikey-footprints:0805
- RV13, RV14, RV15, RV16: footprint (none) -> Potentiometers:Potentiometer_Bourns_PTV09A-1_Horizontal
- U8: footprint (none) -> digikey-footprints:DIP-16_W7.62mm
Changed lines of the file:
@@
 F 0 "U8" H 4850 3300 50  0000 C CNN
 F 1 "PT2399" H 4850 1900 50  0000 C CNN
-F 2 "" H 4850 2200 50  0001 C CNN
+F 2 "digikey-footprints:DIP-16_W7.62mm" H 4850 2200 50  0001 C CNN
 F 3 "" H 4850 2200 50  0001 C CNN
 	1    4850 2600
@@
 F 0 "R57" V 4130 2800 50  0000 C CNN
 F 1 "4.7k" V 4050 2800 50  0000 C CNN
-F 2 "" V 3980 2800 50  0001 C CNN
+F 2 "digikey-footprints:0805" V 3980 2800 50  0001 C CNN
 F 3 "" H 4050 2800 50  0001 C CNN
 	1    4050 2800
@@
 F 0 "RV13" V 3475 2800 50  0000 C CNN
 F 1 "20kA" V 3550 2800 50  0000 C CNN
-F 2 "" H 3650 2800 50  0001 C CNN
+F 2 "Potentiometers:Potentiometer_Bourns_PTV09A-1_Horizontal" H 3650 2800 50  0001 C CNN
 F 3 "" H 3650 2800 50  0001 C CNN
 	1    3650 2800
@@
 F 0 "R67" V 6080 2650 50  0000 C CNN
 F 1 "10k" V 6000 2650 50  0000 C CNN
-F 2 "" V 5930 2650 50  0001 C CNN
+F 2 "digikey-footprints:0805" V 5930 2650 50  0001 C CNN
 F 3 "" H 6000 2650 50  0001 C CNN
 	1    6000 2650
@@
 F 0 "R66" V 6080 2500 50  0000 C CNN
 F 1 "10k" V 6000 2500 50  0000 C CNN
-F 2 "" V 5930 2500 50  0001 C CNN
+F 2 "digikey-footprints:0805" V 5930 2500 50  0001 C CNN
 F 3 "" H 6000 2500 50  0001 C CNN
 	1    6000 2500
@@
 F 0 "R65" V 6080 2350 50  0000 C CNN
 F 1 "15k" V 6000 2350 50  0000 C CNN
-F 2 "" V 5930 2350 50  0001 C CNN
+F 2 "digikey-footprints:0805" V 5930 2350 50  0001 C CNN
 F 3 "" H 6000 2350 50  0001 C CNN
 	1    6000 2350
@@
 F 0 "R71" V 6680 2250 50  0000 C CNN
 F 1 "5.6k" V 6600 2250 50  0000 C CNN
-F 2 "" V 6530 2250 50  0001 C CNN
+F 2 "digikey-footprints:0805" V 6530 2250 50  0001 C CNN
 F 3 "" H 6600 2250 50  0001 C CNN
 	1    6600 2250
@@
 F 0 "RV15" V 7225 2450 50  0000 C CNN
 F 1 "50kA" V 7300 2450 50  0000 C CNN
-F 2 "" H 7400 2450 50  0001 C CNN
+F 2 "Potentiometers:Potentiometer_Bourns_PTV09A-1_Horizontal" H 7400 2450 50  0001 C CNN
 F 3 "" H 7400 2450 50  0001 C CNN
 	1    7400 2450
@@
 F 0 "R73" V 7780 2450 50  0000 C CNN
 F 1 "10k" V 7700 2450 50  0000 C CNN
-F 2 "" V 7630 2450 50  0001 C CNN
+F 2 "digikey-footprints:0805" V 7630 2450 50  0001 C CNN
 F 3 "" H 7700 2450 50  0001 C CNN
 	1    7700 2450
@@
 F 0 "R64" V 6080 2150 50  0000 C CNN
 F 1 "10k" V 6000 2150 50  0000 C CNN
-F 2 "" V 5930 2150 50  0001 C CNN
+F 2 "digikey-footprints:0805" V 5930 2150 50  0001 C CNN
 F 3 "" H 6000 2150 50  0001 C CNN
 	1    6000 2150
@@
 F 0 "R63" V 6080 2000 50  0000 C CNN
 F 1 "10k" V 6000 2000 50  0000 C CNN
-F 2 "" V 5930 2000 50  0001 C CNN
+F 2 "digikey-footprints:0805" V 5930 2000 50  0001 C CNN
 F 3 "" H 6000 2000 50  0001 C CNN
 	1    6000 2000
@@
 F 0 "R70" V 6630 1450 50  0000 C CNN
 F 1 "15k" V 6550 1450 50  0000 C CNN
-F 2 "" V 6480 1450 50  0001 C CNN
+F 2 "digikey-footprints:0805" V 6480 1450 50  0001 C CNN
 F 3 "" H 6550 1450 50  0001 C CNN
 	1    6550 1450
@@
 F 0 "R72" V 7230 1650 50  0000 C CNN
 F 1 "100k" V 7150 1650 50  0000 C CNN
-F 2 "" V 7080 1650 50  0001 C CNN
+F 2 "digikey-footprints:0805" V 7080 1650 50  0001 C CNN
 F 3 "" H 7150 1650 50  0001 C CNN
 	1    7150 1650
@@
 F 0 "R77" V 8630 2100 50  0000 C CNN
 F 1 "4.7k" V 8550 2100 50  0000 C CNN
-F 2 "" V 8480 2100 50  0001 C CNN
+F 2 "digikey-footprints:0805" V 8480 2100 50  0001 C CNN
 F 3 "" H 8550 2100 50  0001 C CNN
 	1    8550 2100
@@
 F 0 "RV16" V 8975 2350 50  0000 C CNN
 F 1 "50kA" V 9050 2350 50  0000 C CNN
-F 2 "" H 9150 2350 50  0001 C CNN
+F 2 "Potentiometers:Potentiometer_Bourns_PTV09A-1_Horizontal" H 9150 2350 50  0001 C CNN
 F 3 "" H 9150 2350 50  0001 C CNN
 	1    9150 2350
@@
 F 0 "RV14" V 4975 4700 50  0000 C CNN
 F 1 "20k" V 5050 4700 50  0000 C CNN
-F 2 "" H 5150 4700 50  0001 C CNN
+F 2 "Potentiometers:Potentiometer_Bourns_PTV09A-1_Horizontal" H 5150 4700 50  0001 C CNN
 F 3 "" H 5150 4700 50  0001 C CNN
 	1    5150 4700
