File: Hardware/Synth Engine/power.sch (KiCad schematic (older format))
At the start: 9 parts, among them J1 Barrel_Jack, U4 TL074, U7 V7805-1000

Commit message: add separate Kicad project for control board. There will now be a separate board for all potentiometers and switches with no other components. Also add connectors between boards.
Parts:
- C18: footprint Capacitors_SMD:CP_Elec_4x4.5 -> digikey-footprints:0805
- C19: footprint Capacitors_SMD:CP_Elec_4x5.7 -> digikey-footprints:0805
Changed lines of the file:
@@
 $EndComp
 $Comp
-L +15V #PWR23
+L +15V #PWR017
 U 1 1 5C3922F5
 P 2700 1500
-F 0 "#PWR23" H 2700 1350 50  0001 C CNN
+F 0 "#PWR017" H 2700 1350 50  0001 C CNN
 F 1 "+15V" H 2700 1640 50  0000 C CNN
 F 2 "" H 2700 1500 50  0001 C CNN
@@
 Check wall wart \npolarity vs DC barrel \njack pinout
 $Comp
-L GND #PWR20
+L GND #PWR018
 U 1 1 5C39231B
 P 2150 1850
-F 0 "#PWR20" H 2150 1600 50  0001 C CNN
+F 0 "#PWR018" H 2150 1600 50  0001 C CNN
 F 1 "GND" H 2150 1700 50  0000 C CNN
 F 2 "" H 2150 1850 50  0001 C CNN
@@
 $EndComp
 $Comp
-L GND #PWR18
+L GND #PWR019
 U 1 1 5C392477
 P 1550 3500
-F 0 "#PWR18" H 1550 3250 50  0001 C CNN
+F 0 "#PWR019" H 1550 3250 50  0001 C CNN
 F 1 "GND" H 1550 3350 50  0000 C CNN
 F 2 "" H 1550 3500 50  0001 C CNN
@@
 $EndComp
 $Comp
-L GND #PWR19
+L GND #PWR020
 U 1 1 5C392498
 P 1900 3500
-F 0 "#PWR19" H 1900 3250 50  0001 C CNN
+F 0 "#PWR020" H 1900 3250 50  0001 C CNN
 F 1 "GND" H 1900 3350 50  0000 C CNN
 F 2 "" H 1900 3500 50  0001 C CNN
@@
 $EndComp
 $Comp
-L +15V #PWR17
+L +15V #PWR021
 U 1 1 5C3924B7
 P 1550 2800
-F 0 "#PWR17" H 1550 2650 50  0001 C CNN
+F 0 "#PWR021" H 1550 2650 50  0001 C CNN
 F 1 "+15V" H 1550 2940 50  0000 C CNN
 F 2 "" H 1550 2800 50  0001 C CNN
@@
 F 0 "C18" H 4710 3020 50  0000 L CNN
 F 1 "0.33uF" H 4710 2870 50  0000 L CNN
-F 2 "Capacitors_SMD:CP_Elec_4x4.5" H 4700 2950 50  0001 C CNN
+F 2 "digikey-footprints:0805" H 4700 2950 50  0001 C CNN
 F 3 "" H 4700 2950 50  0001 C CNN
 	1    4700 2950
@@
 	4700 2750 4950 2750
 $Comp
-L +15V #PWR24
+L +15V #PWR022
 U 1 1 5C392EAE
 P 4700 2650
-F 0 "#PWR24" H 4700 2500 50  0001 C CNN
+F 0 "#PWR022" H 4700 2500 50  0001 C CNN
 F 1 "+15V" H 4700 2790 50  0000 C CNN
 F 2 "" H 4700 2650 50  0001 C CNN
@@
 Connection ~ 4700 2750
 $Comp
-L GND #PWR25
+L GND #PWR023
 U 1 1 5C392EE5
 P 4700 3050
-F 0 "#PWR25" H 4700 2800 50  0001 C CNN
+F 0 "#PWR023" H 4700 2800 50  0001 C CNN
 F 1 "GND" H 4700 2900 50  0000 C CNN
 F 2 "" H 4700 3050 50  0001 C CNN
@@
 $EndComp
 $Comp
-L GND #PWR26
+L GND #PWR024
 U 1 1 5C392F13
 P 5350 3150
-F 0 "#PWR26" H 5350 2900 50  0001 C CNN
+F 0 "#PWR024" H 5350 2900 50  0001 C CNN
 F 1 "GND" H 5350 3000 50  0000 C CNN
 F 2 "" H 5350 3150 50  0001 C CNN
@@
 F 0 "C19" H 5960 3070 50  0000 L CNN
 F 1 "0.1uF" H 5960 2920 50  0000 L CNN
-F 2 "Capacitors_SMD:CP_Elec_4x5.7" H 5950 3000 50  0001 C CNN
+F 2 "digikey-footprints:0805" H 5950 3000 50  0001 C CNN
 F 3 "" H 5950 3000 50  0001 C CNN
 	1    5950 3000
@@
 $EndComp
 $Comp
-L GND #PWR28
+L GND #PWR025
 U 1 1 5C393000
 P 5950 3100
-F 0 "#PWR28" H 5950 2850 50  0001 C CNN
+F 0 "#PWR025" H 5950 2850 50  0001 C CNN
 F 1 "GND" H 5950 2950 50  0000 C CNN
 F 2 "" H 5950 3100 50  0001 C CNN
@@
 $EndComp
 $Comp
-L GND #PWR21
+L GND #PWR026
 U 1 1 5C39BA81
 P 2200 2550
-F 0 "#PWR21" H 2200 2300 50  0001 C CNN
+F 0 "#PWR026" H 2200 2300 50  0001 C CNN
 F 1 "GND" H 2200 2400 50  0000 C CNN
 F 2 "" H 2200 2550 50  0001 C CNN
@@
 $EndComp
 $Comp
-L +15V #PWR22
+L +15V #PWR027
 U 1 1 5C39BAA7
 P 2200 3150
-F 0 "#PWR22" H 2200 3000 50  0001 C CNN
+F 0 "#PWR027" H 2200 3000 50  0001 C CNN
 F 1 "+15V" H 2200 3290 50  0000 C CNN
 F 2 "" H 2200 3150 50  0001 C CNN
@@
 	5950 2600 5950 2900
 $Comp
-L +5V #PWR27
+L +5V #PWR028
 U 1 1 5C548CA8
 P 5950 2600
-F 0 "#PWR27" H 5950 2450 50  0001 C CNN
+F 0 "#PWR028" H 5950 2450 50  0001 C CNN
 F 1 "+5V" H 5950 2740 50  0000 C CNN
 F 2 "" H 5950 2600 50  0001 C CNN
