File: Hardware/Synth Engine/power.sch (KiCad schematic (older format))
At the start: 9 parts, among them J1 Conn_01x02, U4 TL074, U7 V7805-1000

Commit message: arrange reference designators on main board
Parts:
- J1: footprint Connectors_Molex:Molex_KK-6410-02_02x2.54mm_Straight -> Pin_Headers:Pin_Header_Straight_1x02_Pitch2.00mm
Changed lines of the file:
@@
 F 0 "J1" H 1900 1700 50  0000 C CNN
 F 1 "Conn_01x02" H 1900 1400 50  0000 C CNN
-F 2 "Connectors_Molex:Molex_KK-6410-02_02x2.54mm_Straight" H 1900 1600 50  0001 C CNN
+F 2 "Pin_Headers:Pin_Header_Straight_1x02_Pitch2.00mm" H 1900 1600 50  0001 C CNN
 F 3 "" H 1900 1600 50  0001 C CNN
 	1    1900 1600
