File: Hardware/Synth Engine/vca.sch (KiCad schematic (older format))
At the start: 73 parts, among them Q1 MMBT3904-TP, Q2 MMBT3904-TP, Q3 MMBT3904-TP, Q4 MMBT3904-TP, Q5 MMBFJ177, Q6 MMBFJ177, Q7 MMBFJ177, Q8 MMBFJ177, U2 TL074

Commit message: add separate Kicad project for control board. There will now be a separate board for all potentiometers and switches with no other components. Also add connectors between boards.
Parts:
- C20, C21, C22, C23: footprint Capacitors_SMD:CP_Elec_8x10 -> Capacitors_SMD:CP_Elec_4x4.5
- RV5, RV6, RV7, RV8: footprint (none) -> Potentiometers:Potentiometer_Trimmer-EVM3E
