File: Hardware/Synth Engine/vcf.sch (KiCad schematic (older format))
At the start: 37 parts, among them U1 TL074

Commit message: add separate Kicad project for control board. There will now be a separate board for all potentiometers and switches with no other components. Also add connectors between boards.
Parts:
- C10, C11, C12, C5, C6, C7, C8, C9: footprint Capacitors_SMD:CP_Elec_4x4.5 -> digikey-footprints:0805
- RV1, RV2, RV3, RV4: footprint (none) -> Potentiometers:Potentiometer_Trimmer-EVM3E
Changed lines of the file:
@@
 F 0 "C5" H 5310 1970 50  0000 L CNN
 F 1 "10nF" H 5310 1820 50  0000 L CNN
-F 2 "Capacitors_SMD:CP_Elec_4x4.5" H 5300 1900 50  0001 C CNN
+F 2 "digikey-footprints:0805" H 5300 1900 50  0001 C CNN
 F 3 "" H 5300 1900 50  0001 C CNN
 	1    5300 1900
@@
 $EndComp
 $Comp
-L GND #PWR1
+L GND #PWR01
 U 1 1 5C37BDA3
 P 5300 2100
-F 0 "#PWR1" H 5300 1850 50  0001 C CNN
+F 0 "#PWR01" H 5300 1850 50  0001 C CNN
 F 1 "GND" H 5300 1950 50  0000 C CNN
 F 2 "" H 5300 2100 50  0001 C CNN
@@
 $EndComp
 $Comp
-L GND #PWR6
+L GND #PWR02
 U 1 1 5C37D802
 P 5800 2050
-F 0 "#PWR6" H 5800 1800 50  0001 C CNN
+F 0 "#PWR02" H 5800 1800 50  0001 C CNN
 F 1 "GND" H 5800 1900 50  0000 C CNN
 F 2 "" H 5800 2050 50  0001 C CNN
@@
 $EndComp
 $Comp
-L +15V #PWR5
+L +15V #PWR03
 U 1 1 5C38D36B
 P 5800 1450
-F 0 "#PWR5" H 5800 1300 50  0001 C CNN
+F 0 "#PWR03" H 5800 1300 50  0001 C CNN
 F 1 "+15V" H 5800 1590 50  0000 C CNN
 F 2 "" H 5800 1450 50  0001 C CNN
@@
 F 0 "C9" H 5860 1070 50  0000 L CNN
 F 1 "10nF" H 5860 920 50  0000 L CNN
-F 2 "Capacitors_SMD:CP_Elec_4x4.5" H 5850 1000 50  0001 C CNN
+F 2 "digikey-footprints:0805" H 5850 1000 50  0001 C CNN
 F 3 "" H 5850 1000 50  0001 C CNN
 	1    5850 1000
@@
 F 0 "RV1" H 4400 1700 50  0000 C CNN
 F 1 "POT_Dual" H 4400 1625 50  0000 C CNN
-F 2 "" H 4650 1475 50  0001 C CNN
+F 2 "Potentiometers:Potentiometer_Trimmer-EVM3E" H 4650 1475 50  0001 C CNN
 F 3 "" H 4650 1475 50  0001 C CNN
 	1    4400 1550
@@
 $EndComp
 $Comp
-L GND #PWR13
+L GND #PWR04
 U 1 1 5C53B848
 P 6700 2100
-F 0 "#PWR13" H 6700 1850 50  0001 C CNN
+F 0 "#PWR04" H 6700 1850 50  0001 C CNN
 F 1 "GND" H 6700 1950 50  0000 C CNN
 F 2 "" H 6700 2100 50  0001 C CNN
@@
 F 0 "C6" H 5310 3470 50  0000 L CNN
 F 1 "10nF" H 5310 3320 50  0000 L CNN
-F 2 "Capacitors_SMD:CP_Elec_4x4.5" H 5300 3400 50  0001 C CNN
+F 2 "digikey-footprints:0805" H 5300 3400 50  0001 C CNN
 F 3 "" H 5300 3400 50  0001 C CNN
 	1    5300 3400
@@
 $EndComp
 $Comp
-L GND #PWR2
+L GND #PWR05
 U 1 1 5C53C629
 P 5300 3600
-F 0 "#PWR2" H 5300 3350 50  0001 C CNN
+F 0 "#PWR05" H 5300 3350 50  0001 C CNN
 F 1 "GND" H 5300 3450 50  0000 C CNN
 F 2 "" H 5300 3600 50  0001 C CNN
@@
 $EndComp
 $Comp
-L GND #PWR8
+L GND #PWR06
 U 1 1 5C53C63B
 P 5800 3550
-F 0 "#PWR8" H 5800 3300 50  0001 C CNN
+F 0 "#PWR06" H 5800 3300 50  0001 C CNN
 F 1 "GND" H 5800 3400 50  0000 C CNN
 F 2 "" H 5800 3550 50  0001 C CNN
@@
 $EndComp
 $Comp
-L +15V #PWR7
+L +15V #PWR07
 U 1 1 5C53C641
 P 5800 2950
-F 0 "#PWR7" H 5800 2800 50  0001 C CNN
+F 0 "#PWR07" H 5800 2800 50  0001 C CNN
 F 1 "+15V" H 5800 3090 50  0000 C CNN
 F 2 "" H 5800 2950 50  0001 C CNN
@@
 F 0 "C10" H 5860 2570 50  0000 L CNN
 F 1 "10nF" H 5860 2420 50  0000 L CNN
-F 2 "Capacitors_SMD:CP_Elec_4x4.5" H 5850 2500 50  0001 C CNN
+F 2 "digikey-footprints:0805" H 5850 2500 50  0001 C CNN
 F 3 "" H 5850 2500 50  0001 C CNN
 	1    5850 2500
@@
 F 0 "RV2" H 4400 3200 50  0000 C CNN
 F 1 "POT_Dual" H 4400 3125 50  0000 C CNN
-F 2 "" H 4650 2975 50  0001 C CNN
+F 2 "Potentiometers:Potentiometer_Trimmer-EVM3E" H 4650 2975 50  0001 C CNN
 F 3 "" H 4650 2975 50  0001 C CNN
 	1    4400 3050
@@
 $EndComp
 $Comp
-L GND #PWR14
+L GND #PWR08
 U 1 1 5C53C691
 P 6700 3600
-F 0 "#PWR14" H 6700 3350 50  0001 C CNN
+F 0 "#PWR08" H 6700 3350 50  0001 C CNN
 F 1 "GND" H 6700 3450 50  0000 C CNN
 F 2 "" H 6700 3600 50  0001 C CNN
@@
 F 0 "C7" H 5310 4920 50  0000 L CNN
 F 1 "10nF" H 5310 4770 50  0000 L CNN
-F 2 "Capacitors_SMD:CP_Elec_4x4.5" H 5300 4850 50  0001 C CNN
+F 2 "digikey-footprints:0805" H 5300 4850 50  0001 C CNN
 F 3 "" H 5300 4850 50  0001 C CNN
 	1    5300 4850
@@
 $EndComp
 $Comp
-L GND #PWR3
+L GND #PWR09
 U 1 1 5C53CB2F
 P 5300 5050
-F 0 "#PWR3" H 5300 4800 50  0001 C CNN
+F 0 "#PWR09" H 5300 4800 50  0001 C CNN
 F 1 "GND" H 5300 4900 50  0000 C CNN
 F 2 "" H 5300 5050 50  0001 C CNN
@@
 $EndComp
 $Comp
-L GND #PWR10
+L GND #PWR010
 U 1 1 5C53CB41
 P 5800 5000
-F 0 "#PWR10" H 5800 4750 50  0001 C CNN
+F 0 "#PWR010" H 5800 4750 50  0001 C CNN
 F 1 "GND" H 5800 4850 50  0000 C CNN
 F 2 "" H 5800 5000 50  0001 C CNN
@@
 $EndComp
 $Comp
-L +15V #PWR9
+L +15V #PWR011
 U 1 1 5C53CB47
 P 5800 4400
-F 0 "#PWR9" H 5800 4250 50  0001 C CNN
+F 0 "#PWR011" H 5800 4250 50  0001 C CNN
 F 1 "+15V" H 5800 4540 50  0000 C CNN
 F 2 "" H 5800 4400 50  0001 C CNN
@@
 F 0 "C11" H 5860 4020 50  0000 L CNN
 F 1 "10nF" H 5860 3870 50  0000 L CNN
-F 2 "Capacitors_SMD:CP_Elec_4x4.5" H 5850 3950 50  0001 C CNN
+F 2 "digikey-footprints:0805" H 5850 3950 50  0001 C CNN
 F 3 "" H 5850 3950 50  0001 C CNN
 	1    5850 3950
@@
 F 0 "RV3" H 4400 4650 50  0000 C CNN
 F 1 "POT_Dual" H 4400 4575 50  0000 C CNN
-F 2 "" H 4650 4425 50  0001 C CNN
+F 2 "Potentiometers:Potentiometer_Trimmer-EVM3E" H 4650 4425 50  0001 C CNN
 F 3 "" H 4650 4425 50  0001 C CNN
 	1    4400 4500
@@
 $EndComp
 $Comp
-L GND #PWR15
+L GND #PWR012
 U 1 1 5C53CB97
 P 6700 5050
-F 0 "#PWR15" H 6700 4800 50  0001 C CNN
+F 0 "#PWR012" H 6700 4800 50  0001 C CNN
 F 1 "GND" H 6700 4900 50  0000 C CNN
 F 2 "" H 6700 5050 50  0001 C CNN
@@
 F 0 "C8" H 5310 6420 50  0000 L CNN
 F 1 "10nF" H 5310 6270 50  0000 L CNN
-F 2 "Capacitors_SMD:CP_Elec_4x4.5" H 5300 6350 50  0001 C CNN
+F 2 "digikey-footprints:0805" H 5300 6350 50  0001 C CNN
 F 3 "" H 5300 6350 50  0001 C CNN
 	1    5300 6350
@@
 $EndComp
 $Comp
-L GND #PWR4
+L GND #PWR013
 U 1 1 5C53CBAD
 P 5300 6550
-F 0 "#PWR4" H 5300 6300 50  0001 C CNN
+F 0 "#PWR013" H 5300 6300 50  0001 C CNN
 F 1 "GND" H 5300 6400 50  0000 C CNN
 F 2 "" H 5300 6550 50  0001 C CNN
@@
 $EndComp
 $Comp
-L GND #PWR12
+L GND #PWR014
 U 1 1 5C53CBBF
 P 5800 6500
-F 0 "#PWR12" H 5800 6250 50  0001 C CNN
+F 0 "#PWR014" H 5800 6250 50  0001 C CNN
 F 1 "GND" H 5800 6350 50  0000 C CNN
 F 2 "" H 5800 6500 50  0001 C CNN
@@
 $EndComp
 $Comp
-L +15V #PWR11
+L +15V #PWR015
 U 1 1 5C53CBC5
 P 5800 5900
-F 0 "#PWR11" H 5800 5750 50  0001 C CNN
+F 0 "#PWR015" H 5800 5750 50  0001 C CNN
 F 1 "+15V" H 5800 6040 50  0000 C CNN
 F 2 "" H 5800 5900 50  0001 C CNN
@@
 F 0 "C12" H 5860 5520 50  0000 L CNN
 F 1 "10nF" H 5860 5370 50  0000 L CNN
-F 2 "Capacitors_SMD:CP_Elec_4x4.5" H 5850 5450 50  0001 C CNN
+F 2 "digikey-footprints:0805" H 5850 5450 50  0001 C CNN
 F 3 "" H 5850 5450 50  0001 C CNN
 	1    5850 5450
@@
 F 0 "RV4" H 4400 6150 50  0000 C CNN
 F 1 "POT_Dual" H 4400 6075 50  0000 C CNN
-F 2 "" H 4650 5925 50  0001 C CNN
+F 2 "Potentiometers:Potentiometer_Trimmer-EVM3E" H 4650 5925 50  0001 C CNN
 F 3 "" H 4650 5925 50  0001 C CNN
 	1    4400 6000
@@
 $EndComp
 $Comp
-L GND #PWR16
+L GND #PWR016
 U 1 1 5C53CC15
 P 6700 6550
-F 0 "#PWR16" H 6700 6300 50  0001 C CNN
+F 0 "#PWR016" H 6700 6300 50  0001 C CNN
 F 1 "GND" H 6700 6400 50  0000 C CNN
 F 2 "" H 6700 6550 50  0001 C CNN
