File: Hardware/Synth Engine/vcf.sch (KiCad schematic (older format))
At the start: 37 parts, among them U1 TL074

Commit message: connect control board to main synth schem pages
Parts:
- removed RV1, RV2, RV3, RV4: POT_Dual, Potentiometers:Potentiometer_Trimmer-EVM3E, symbol POT_Dual
Connections:
- net labels added: freq_fb_1, freq_fb_2, freq_fb_3, freq_fb_4, freq_in_1, freq_in_2, freq_in_3, freq_in_4, freq_out_1, freq_out_2, freq_out_3, freq_out_4
- wire segments 104 -> 76
Other:
- moved on the sheet: C1, C2, C3, C4, R1, R2, R3, R4
Changed lines of the file:
@@
 Comment4 ""
 $EndDescr
-Text HLabel 3100 1650 0    60   Input ~ 0
+Text HLabel 2750 1650 0    60   Input ~ 0
 osc1
-Text HLabel 3100 3150 0    60   Input ~ 0
+Text HLabel 2750 3150 0    60   Input ~ 0
 osc2
-Text HLabel 3100 4600 0    60   Input ~ 0
+Text HLabel 2750 4600 0    60   Input ~ 0
 osc3
-Text HLabel 3100 6100 0    60   Input ~ 0
+Text HLabel 2750 6100 0    60   Input ~ 0
 osc4
 Text HLabel 6800 1750 2    60   Input ~ 0
@@
 L CP1_Small C1
 U 1 1 5C37CAF6
-P 3350 1650
-F 0 "C1" H 3360 1720 50  0000 L CNN
-F 1 "22uF" H 3360 1570 50  0000 L CNN
-F 2 "Capacitors_SMD:CP_Elec_5x5.7" H 3350 1650 50  0001 C CNN
-F 3 "" H 3350 1650 50  0001 C CNN
-	1    3350 1650
+P 3000 1650
+F 0 "C1" H 3010 1720 50  0000 L CNN
+F 1 "22uF" H 3010 1570 50  0000 L CNN
+F 2 "Capacitors_SMD:CP_Elec_5x5.7" H 3000 1650 50  0001 C CNN
+F 3 "" H 3000 1650 50  0001 C CNN
+	1    3000 1650
 	0    1    1    0
 $EndComp
@@
 L R R1
 U 1 1 5C537DA0
-P 3700 1650
-F 0 "R1" V 3780 1650 50  0000 C CNN
-F 1 "1k" V 3700 1650 50  0000 C CNN
-F 2 "digikey-footprints:0805" V 3630 1650 50  0001 C CNN
-F 3 "" H 3700 1650 50  0001 C CNN
-	1    3700 1650
+P 3350 1650
+F 0 "R1" V 3430 1650 50  0000 C CNN
+F 1 "1k" V 3350 1650 50  0000 C CNN
+F 2 "digikey-footprints:0805" V 3280 1650 50  0001 C CNN
+F 3 "" H 3350 1650 50  0001 C CNN
+	1    3350 1650
 	0    1    1    0
 $EndComp
@@
 	0    1    1    0
 $EndComp
-$Comp
-L POT_Dual RV1
-U 1 1 5C53920C
-P 4400 1550
-F 0 "RV1" H 4400 1700 50  0000 C CNN
-F 1 "POT_Dual" H 4400 1625 50  0000 C CNN
-F 2 "Potentiometers:Potentiometer_Trimmer-EVM3E" H 4650 1475 50  0001 C CNN
-F 3 "" H 4650 1475 50  0001 C CNN
-	1    4400 1550
-	1    0    0    -1
-$EndComp
-Connection ~ 4450 1400
-Wire Wire Line
-	4650 1400 4450 1400
-Connection ~ 4450 1650
-Wire Wire Line
-	4450 1000 4450 1650
 Wire Wire Line
 	4800 1650 4950 1650
 Wire Wire Line
-	4650 1450 4650 1400
-Wire Wire Line
-	4300 1650 4500 1650
-Wire Wire Line
-	3250 1650 3100 1650
+	2900 1650 2750 1650
 Connection ~ 5300 1650
 Wire Wire Line
 	5300 1800 5300 1650
 Wire Wire Line
-	3550 1650 3450 1650
+	3200 1650 3100 1650
 Wire Wire Line
 	4450 1000 5750 1000
@@
 	5450 1850 5600 1850
 Wire Wire Line
-	4150 1450 4150 1400
-Wire Wire Line
-	4150 1400 3900 1400
-Wire Wire Line
-	3900 1400 3900 1650
-Wire Wire Line
-	3850 1650 4000 1650
-Connection ~ 3900 1650
+	3500 1650 3650 1650
 $Comp
 L CP1_Small C13
@@
 L CP1_Small C2
 U 1 1 5C53C635
-P 3350 3150
-F 0 "C2" H 3360 3220 50  0000 L CNN
-F 1 "22uF" H 3360 3070 50  0000 L CNN
-F 2 "Capacitors_SMD:CP_Elec_5x5.7" H 3350 3150 50  0001 C CNN
-F 3 "" H 3350 3150 50  0001 C CNN
-	1    3350 3150
+P 3000 3150
+F 0 "C2" H 3010 3220 50  0000 L CNN
+F 1 "22uF" H 3010 3070 50  0000 L CNN
+F 2 "Capacitors_SMD:CP_Elec_5x5.7" H 3000 3150 50  0001 C CNN
+F 3 "" H 3000 3150 50  0001 C CNN
+	1    3000 3150
 	0    1    1    0
 $EndComp
@@
 L R R2
 U 1 1 5C53C648
-P 3700 3150
-F 0 "R2" V 3780 3150 50  0000 C CNN
-F 1 "1k" V 3700 3150 50  0000 C CNN
-F 2 "digikey-footprints:0805" V 3630 3150 50  0001 C CNN
-F 3 "" H 3700 3150 50  0001 C CNN
-	1    3700 3150
+P 3350 3150
+F 0 "R2" V 3430 3150 50  0000 C CNN
+F 1 "1k" V 3350 3150 50  0000 C CNN
+F 2 "digikey-footprints:0805" V 3280 3150 50  0001 C CNN
+F 3 "" H 3350 3150 50  0001 C CNN
+	1    3350 3150
 	0    1    1    0
 $EndComp
@@
 	0    1    1    0
 $EndComp
-$Comp
-L POT_Dual RV2
-U 1 1 5C53C65A
-P 4400 3050
-F 0 "RV2" H 4400 3200 50  0000 C CNN
-F 1 "POT_Dual" H 4400 3125 50  0000 C CNN
-F 2 "Potentiometers:Potentiometer_Trimmer-EVM3E" H 4650 2975 50  0001 C CNN
-F 3 "" H 4650 2975 50  0001 C CNN
-	1    4400 3050
-	1    0    0    -1
-$EndComp
-Connection ~ 4450 2900
-Wire Wire Line
-	4650 2900 4450 2900
-Connection ~ 4450 3150
-Wire Wire Line
-	4450 2500 4450 3150
 Wire Wire Line
 	4800 3150 4950 3150
 Wire Wire Line
-	4650 2950 4650 2900
-Wire Wire Line
-	4300 3150 4500 3150
-Wire Wire Line
-	3250 3150 3100 3150
+	2900 3150 2750 3150
 Connection ~ 5300 3150
 Wire Wire Line
 	5300 3300 5300 3150
 Wire Wire Line
-	3550 3150 3450 3150
+	3200 3150 3100 3150
 Wire Wire Line
 	4450 2500 5750 2500
@@
 	5450 3350 5600 3350
 Wire Wire Line
-	4150 2950 4150 2900
-Wire Wire Line
-	4150 2900 3900 2900
-Wire Wire Line
-	3900 2900 3900 3150
-Wire Wire Line
-	3850 3150 4000 3150
-Connection ~ 3900 3150
+	3500 3150 3650 3150
 $Comp
 L CP1_Small C14
@@
 L CP1_Small C3
 U 1 1 5C53CB3B
-P 3350 4600
-F 0 "C3" H 3360 4670 50  0000 L CNN
-F 1 "22uF" H 3360 4520 50  0000 L CNN
-F 2 "Capacitors_SMD:CP_Elec_5x5.7" H 3350 4600 50  0001 C CNN
-F 3 "" H 3350 4600 50  0001 C CNN
-	1    3350 4600
+P 3000 4600
+F 0 "C3" H 3010 4670 50  0000 L CNN
+F 1 "22uF" H 3010 4520 50  0000 L CNN
+F 2 "Capacitors_SMD:CP_Elec_5x5.7" H 3000 4600 50  0001 C CNN
+F 3 "" H 3000 4600 50  0001 C CNN
+	1    3000 4600
 	0    1    1    0
 $EndComp
@@
 L R R3
 U 1 1 5C53CB4E
-P 3700 4600
-F 0 "R3" V 3780 4600 50  0000 C CNN
-F 1 "1k" V 3700 4600 50  0000 C CNN
-F 2 "digikey-footprints:0805" V 3630 4600 50  0001 C CNN
-F 3 "" H 3700 4600 50  0001 C CNN
-	1    3700 4600
+P 3350 4600
+F 0 "R3" V 3430 4600 50  0000 C CNN
+F 1 "1k" V 3350 4600 50  0000 C CNN
+F 2 "digikey-footprints:0805" V 3280 4600 50  0001 C CNN
+F 3 "" H 3350 4600 50  0001 C CNN
+	1    3350 4600
 	0    1    1    0
 $EndComp
@@
 	0    1    1    0
 $EndComp
-$Comp
-L POT_Dual RV3
-U 1 1 5C53CB60
-P 4400 4500
-F 0 "RV3" H 4400 4650 50  0000 C CNN
-F 1 "POT_Dual" H 4400 4575 50  0000 C CNN
-F 2 "Potentiometers:Potentiometer_Trimmer-EVM3E" H 4650 4425 50  0001 C CNN
-F 3 "" H 4650 4425 50  0001 C CNN
-	1    4400 4500
-	1    0    0    -1
-$EndComp
-Connection ~ 4450 4350
-Wire Wire Line
-	4650 4350 4450 4350
-Connection ~ 4450 4600
-Wire Wire Line
-	4450 3950 4450 4600
 Wire Wire Line
 	4800 4600 4950 4600
 Wire Wire Line
-	4650 4400 4650 4350
-Wire Wire Line
-	4300 4600 4500 4600
-Wire Wire Line
-	3250 4600 3100 4600
+	2900 4600 2750 4600
 Connection ~ 5300 4600
 Wire Wire Line
 	5300 4750 5300 4600
 Wire Wire Line
-	3550 4600 3450 4600
+	3200 4600 3100 4600
 Wire Wire Line
 	4450 3950 5750 3950
@@
 	5450 4800 5600 4800
 Wire Wire Line
-	4150 4400 4150 4350
-Wire Wire Line
-	4150 4350 3900 4350
-Wire Wire Line
-	3900 4350 3900 4600
-Wire Wire Line
-	3850 4600 4000 4600
-Connection ~ 3900 4600
+	3500 4600 3650 4600
 $Comp
 L CP1_Small C15
@@
 L CP1_Small C4
 U 1 1 5C53CBB9
-P 3350 6100
-F 0 "C4" H 3360 6170 50  0000 L CNN
-F 1 "22uF" H 3360 6020 50  0000 L CNN
-F 2 "Capacitors_SMD:CP_Elec_5x5.7" H 3350 6100 50  0001 C CNN
-F 3 "" H 3350 6100 50  0001 C CNN
-	1    3350 6100
+P 3000 6100
+F 0 "C4" H 3010 6170 50  0000 L CNN
+F 1 "22uF" H 3010 6020 50  0000 L CNN
+F 2 "Capacitors_SMD:CP_Elec_5x5.7" H 3000 6100 50  0001 C CNN
+F 3 "" H 3000 6100 50  0001 C CNN
+	1    3000 6100
 	0    1    1    0
 $EndComp
@@
 L R R4
 U 1 1 5C53CBCC
-P 3700 6100
-F 0 "R4" V 3780 6100 50  0000 C CNN
-F 1 "1k" V 3700 6100 50  0000 C CNN
-F 2 "digikey-footprints:0805" V 3630 6100 50  0001 C CNN
-F 3 "" H 3700 6100 50  0001 C CNN
-	1    3700 6100
+P 3350 6100
+F 0 "R4" V 3430 6100 50  0000 C CNN
+F 1 "1k" V 3350 6100 50  0000 C CNN
+F 2 "digikey-footprints:0805" V 3280 6100 50  0001 C CNN
+F 3 "" H 3350 6100 50  0001 C CNN
+	1    3350 6100
 	0    1    1    0
 $EndComp
@@
 	0    1    1    0
 $EndComp
-$Comp
-L POT_Dual RV4
-U 1 1 5C53CBDE
-P 4400 6000
-F 0 "RV4" H 4400 6150 50  0000 C CNN
-F 1 "POT_Dual" H 4400 6075 50  0000 C CNN
-F 2 "Potentiometers:Potentiometer_Trimmer-EVM3E" H 4650 5925 50  0001 C CNN
-F 3 "" H 4650 5925 50  0001 C CNN
-	1    4400 6000
-	1    0    0    -1
-$EndComp
-Connection ~ 4450 5850
-Wire Wire Line
-	4650 5850 4450 5850
-Connection ~ 4450 6100
-Wire Wire Line
-	4450 5450 4450 6100
 Wire Wire Line
 	4800 6100 4950 6100
 Wire Wire Line
-	4650 5900 4650 5850
-Wire Wire Line
-	4300 6100 4500 6100
-Wire Wire Line
-	3250 6100 3100 6100
+	2900 6100 2750 6100
 Connection ~ 5300 6100
 Wire Wire Line
 	5300 6250 5300 6100
 Wire Wire Line
-	3550 6100 3450 6100
+	3200 6100 3100 6100
 Wire Wire Line
 	4450 5450 5750 5450
@@
 	5450 6300 5600 6300
 Wire Wire Line
-	4150 5900 4150 5850
-Wire Wire Line
-	4150 5850 3900 5850
-Wire Wire Line
-	3900 5850 3900 6100
-Wire Wire Line
-	3850 6100 4000 6100
-Connection ~ 3900 6100
+	3500 6100 3650 6100
 $Comp
 L CP1_Small C16
@@
 	6700 6250 6700 6200
 Connection ~ 6700 6200
+Text HLabel 3650 1650 2    60   Output ~ 0
+freq_in_1
+Text HLabel 4450 1000 0    60   Output ~ 0
+freq_fb_1
+Text HLabel 4800 1650 0    60   Input ~ 0
+freq_out_1
+Text HLabel 3650 3150 2    60   Output ~ 0
+freq_in_2
+Text HLabel 4450 2500 0    60   Output ~ 0
+freq_fb_2
+Text HLabel 4800 3150 0    60   Input ~ 0
+freq_out_2
+Text HLabel 3650 4600 2    60   Output ~ 0
+freq_in_3
+Text HLabel 4450 3950 0    60   Output ~ 0
+freq_fb_3
+Text HLabel 4800 4600 0    60   Input ~ 0
+freq_out_3
+Text HLabel 3650 6100 2    60   Output ~ 0
+freq_in_4
+Text HLabel 4450 5450 0    60   Output ~ 0
+freq_fb_4
+Text HLabel 4800 6100 0    60   Input ~ 0
+freq_out_4
 $EndSCHEMATC

Commit message: route connectors on control board. Will add additional set of connectors for filter knobs to simplify routing.
Connections:
- net at C13.1, C9.1: now also U1.6 (-), U1.7; no longer U1.1, U1.2 (-)
- net at C5.1, R5.1, R9.2: now also U1.5 (+); no longer U1.3 (+)
- net at C6.1, R10.2, R6.1: now also U1.3 (+); no longer U1.5 (+)
- net at C10.1, C14.1: now also U1.1, U1.2 (-); no longer U1.6 (-), U1.7
- net at C7.1, R11.2, R7.1: now also U1.12 (+); no longer U1.10 (+)
- net at C11.1, C15.1: now also U1.13 (-), U1.14; no longer U1.8, U1.9 (-)
- net at C8.1, R12.2, R8.1: now also U1.10 (+); no longer U1.12 (+)
- net at C12.1, C16.1: now also U1.8, U1.9 (-); no longer U1.13 (-), U1.14
Changed lines of the file:
@@
 $Comp
 L TL074 U1
-U 1 1 5C37B428
+U 2 1 5C37B428
 P 5900 1750
 F 0 "U1" H 5900 1950 50  0000 L CNN
@@
 F 2 "digikey-footprints:SOIC-14_W3.9mm" H 5850 1850 50  0001 C CNN
 F 3 "" H 5950 1950 50  0001 C CNN
-	1    5900 1750
+	2    5900 1750
 	1    0    0    -1
 $EndComp
@@
 $Comp
 L TL074 U1
-U 2 1 5C53C61D
+U 1 1 5C53C61D
 P 5900 3250
 F 0 "U1" H 5900 3450 50  0000 L CNN
@@
 F 2 "digikey-footprints:SOIC-14_W3.9mm" H 5850 3350 50  0001 C CNN
 F 3 "" H 5950 3450 50  0001 C CNN
-	2    5900 3250
+	1    5900 3250
 	1    0    0    -1
 $EndComp
@@
 $Comp
 L TL074 U1
-U 3 1 5C53CB23
+U 4 1 5C53CB23
 P 5900 4700
 F 0 "U1" H 5900 4900 50  0000 L CNN
@@
 F 2 "digikey-footprints:SOIC-14_W3.9mm" H 5850 4800 50  0001 C CNN
 F 3 "" H 5950 4900 50  0001 C CNN
-	3    5900 4700
+	4    5900 4700
 	1    0    0    -1
 $EndComp
@@
 $Comp
 L TL074 U1
-U 4 1 5C53CBA1
+U 3 1 5C53CBA1
 P 5900 6200
 F 0 "U1" H 5900 6400 50  0000 L CNN
@@
 F 2 "digikey-footprints:SOIC-14_W3.9mm" H 5850 6300 50  0001 C CNN
 F 3 "" H 5950 6400 50  0001 C CNN
-	4    5900 6200
-	1    0    0    -1
-$EndComp
+	3    5900 6200
+	1    0    0    -1
+$EndComp
