File: Hardware/Synth Engine/synth_psoc.kicad_pcb (KiCad board)
At the start: 2 copper layers, 283 parts, among them J1 Barrel_Jack, J2 Audio-Jack-2_Switch, J3 SWD_programming, J4 Capsense_0, J5 Capsense_1, J6 Capsense_2, J7 Capsense_3, Q1 MMBT3904-TP, Q2 MMBT3904-TP, Q3 MMBT3904-TP, Q4 MMBT3904-TP, Q5 MMBFJ177, Q6 MMBFJ177, Q7 MMBFJ177, Q8 MMBFJ177, SW1 SW_DPDT_x2, SW10 SW_SPST, SW11 SW_SPST, SW12 SW_SPST, SW13 SW_SPST, SW2 SW_SPST, SW3 SW_SPST, SW4 SW_SPST, SW5 SW_SPST, SW6 SW_SPST, SW7 SW_SPST, SW8 SW_SPST, SW9 SW_SPST, U1 TL074, U2 TL074, U3 TL074, U4 TL074, U5 TL074, U6 CY8C4246AZI-L445, U7 V7805-1000, U8 PT2399, Y1 Crystal

Commit message: place MCU footprints
Parts:
- removed J4: Capsense_0, Cypress_capsense:Capsense_button
- removed J5: Capsense_1, Cypress_capsense:Capsense_button
- removed J6: Capsense_2, Cypress_capsense:Capsense_button
- removed J7: Capsense_3, Cypress_capsense:Capsense_button
- removed R103, R104, R105, R106, R107, R108, R109, R110, R115, R116, R117, R118: R, digikey-footprints:0805
- removed RV1, RV2, RV3, RV4: POT_Dual, Potentiometers:Potentiometer_Trimmer-EVM3E
- removed RV10, RV11, RV12, RV9: 100kA, Potentiometers:Potentiometer_Bourns_PTV09A-1_Horizontal
- removed RV17: 10kA, Potentiometers:Potentiometer_Bourns_PTV09A-1_Horizontal
- removed RV22, RV23, RV24, RV25, RV26, RV27, RV28, RV29: 20kA, Potentiometers:Potentiometer_Bourns_PTV09A-1_Horizontal
- removed RV30, RV31, RV32, RV33: 20kB, Potentiometers:Potentiometer_Bourns_PTV09A-1_Horizontal
- removed SW1: SW_DPDT_x2, SparkFun-Electromechanical:SWITCH-SPDT
- removed SW10, SW11, SW12, SW13, SW2, SW3, SW4, SW5, SW6, SW7, SW8, SW9: SW_SPST, SparkFun-Electromechanical:SWITCH-SPDT
- C78, C79, C83, C86, C88: footprint Capacitors_SMD:CP_Elec_4x4.5 -> digikey-footprints:0805
- moved R18 315.2 mm to (68.9, 23.9)
- moved C18 296.3 mm to (69.5, 29.7)
- moved D1 291.7 mm to (62.5, 25.0)
- moved C17 291.7 mm to (92.7, 14.0)
- moved J1 291.7 mm to (72.5, 14.1)
- moved U7 291.7 mm to (78.4, 11.7)
- moved U4 290.6 mm to (94.2, 24.5)
- moved R17 287.3 mm to (76.9, 23.6)
- moved R101 278.6 mm to (19.8, 170.7), turned to 180 degrees
- moved C19 278.4 mm to (80.8, 30.2)
- moved J3 264.0 mm to (64.0, 192.0), turned to 270 degrees
- moved R102 263.5 mm to (19.8, 168.1), turned to 180 degrees
- moved R111 261.9 mm to (64.6, 162.6), turned to 270 degrees
- moved R114 256.0 mm to (58.4, 162.6), turned to 270 degrees
- moved C78 242.7 mm to (48.8, 178.8), turned to 90 degrees
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Connections:
- net /Microcontroller/osc1_quant renamed /Connectors/osc1_quant
- net /Microcontroller/osc1_repeat renamed /Connectors/osc1_repeat
- net /Microcontroller/osc2_quant renamed /Connectors/osc2_quant
- net /Microcontroller/osc2_repeat renamed /Connectors/osc2_repeat
- net /Microcontroller/osc3_quant renamed /Connectors/osc3_quant
- net /Microcontroller/osc3_repeat renamed /Connectors/osc3_repeat
- net /Microcontroller/osc4_quant renamed /Connectors/osc4_quant
- net /Microcontroller/osc4_repeat renamed /Connectors/osc4_repeat
- net Net-(C72-Pad1) renamed /LFO Modulation and Routing/LFO_freq_out
- net Net-(R5-Pad2) renamed /Connectors/freq_out_1
- net Net-(R6-Pad2) renamed /Connectors/freq_out_2
- net Net-(R7-Pad2) renamed /Connectors/freq_out_3
- net Net-(R8-Pad2) renamed /Connectors/freq_out_4
- C10 pad 2: Net-(C10-Pad2) -> /Connectors/freq_fb_2
- C11 pad 2: Net-(C11-Pad2) -> /Connectors/freq_fb_3
- C12 pad 2: Net-(C12-Pad2) -> /Connectors/freq_fb_4
- C9 pad 2: Net-(C9-Pad2) -> /Connectors/freq_fb_1
- R1 pad 1: Net-(R1-Pad1) -> /Connectors/freq_in_1
- R111 pad 2: /Microcontroller/envelope_pwm_1 -> /Connectors/envelope_pwm_bypass_in_1
- R112 pad 2: /Microcontroller/envelope_pwm_2 -> /Connectors/envelope_pwm_bypass_in_2
- R113 pad 2: /Microcontroller/envelope_pwm_3 -> /Connectors/envelope_pwm_bypass_in_3
- R114 pad 2: /Microcontroller/envelope_pwm_4 -> /Connectors/envelope_pwm_bypass_in_4
- R2 pad 1: Net-(R2-Pad1) -> /Connectors/freq_in_2
- R3 pad 1: Net-(R3-Pad1) -> /Connectors/freq_in_3
- R4 pad 1: Net-(R4-Pad1) -> /Connectors/freq_in_4
- R82 pad 1: Net-(R82-Pad1) -> /LFO Modulation and Routing/LFO_freq_in
- U6 pad 1: /Microcontroller/osc1_speed -> /Connectors/osc1_speed
- U6 pad 2: /Microcontroller/osc1_freq_wiper -> /Connectors/osc1_freq_wiper
- U6 pad 3: /Microcontroller/osc1_pwm_wiper -> /Connectors/osc1_pwm_wiper
- U6 pad 4: /Microcontroller/osc2_freq_wiper -> /Connectors/osc2_freq_wiper
- U6 pad 5: /Microcontroller/osc2_pwm_wiper -> /Connectors/osc2_pwm_wiper
- U6 pad 51: /Microcontroller/envelope_pwm_1 -> /Connectors/envelope_pwm_bypass_in_1
- U6 pad 52: /Microcontroller/envelope_pwm_2 -> /Connectors/envelope_pwm_bypass_in_2
- U6 pad 53: /Microcontroller/envelope_pwm_3 -> /Connectors/envelope_pwm_bypass_in_3
- U6 pad 54: /Microcontroller/envelope_pwm_4 -> /Connectors/envelope_pwm_bypass_in_4
- U6 pad 6: /Microcontroller/osc3_freq_wiper -> /Connectors/osc3_freq_wiper
- U6 pad 62: /Microcontroller/osc4_speed -> /Connectors/osc4_speed
- U6 pad 63: /Microcontroller/osc3_speed -> /Connectors/osc3_speed
- U6 pad 64: /Microcontroller/osc2_speed -> /Connectors/osc2_speed
- U6 pad 7: /Microcontroller/osc3_pwm_wiper -> /Connectors/osc3_pwm_wiper
- U6 pad 8: /Microcontroller/osc4_freq_wiper -> /Connectors/osc4_freq_wiper
- U6 pad 9: /Microcontroller/osc4_pwm_wiper -> /Connectors/osc4_pwm_wiper

Commit message: place delay and output mixer footprints
Parts:
- added J10: Conn_01x13, Pin_Headers:Pin_Header_Straight_1x13_Pitch2.54mm, F.Cu at (111.8, 160.5)
- added J11: Conn_01x13, Pin_Headers:Pin_Header_Straight_1x13_Pitch2.54mm, F.Cu at (116.8, 160.5)
- added J4: Conn_01x08, Pin_Headers:Pin_Header_Straight_1x08_Pitch2.54mm, F.Cu at (93.0, 46.7)
- added J5: Conn_01x02, Pin_Headers:Pin_Header_Straight_1x02_Pitch2.54mm, F.Cu at (86.4, 139.2)
- added J6: Conn_01x03, Pin_Headers:Pin_Header_Straight_1x03_Pitch2.54mm, F.Cu at (91.4, 129.5)
- added J7: Capsense_buttons, Pin_Headers:Pin_Header_Straight_1x04_Pitch2.54mm, F.Cu at (67.1, 181.9)
- added J8: Conn_01x13, Pin_Headers:Pin_Header_Straight_1x13_Pitch2.54mm, F.Cu at (101.6, 160.5)
- added J9: Conn_01x13, Pin_Headers:Pin_Header_Straight_1x13_Pitch2.54mm, F.Cu at (106.7, 160.5)
- moved R51 223.0 mm to (100.1, 34.5), turned to 270 degrees
- moved R58 214.2 mm to (103.5, 24.6), turned to 180 degrees
- moved R75 208.1 mm to (109.7, 22.4), turned to 90 degrees
- moved R60 207.1 mm to (115.8, 18.3), turned to 90 degrees
- moved R79 202.6 mm to (99.6, 19.8), turned to 90 degrees
- moved R74 202.3 mm to (107.7, 22.4), turned to 90 degrees
- moved R55 199.4 mm to (112.4, 34.6), turned to 270 degrees
- moved R56 196.1 mm to (109.3, 33.5)
- moved R53 194.6 mm to (104.1, 34.5), turned to 270 degrees
- moved R59 194.3 mm to (118.9, 28.4), turned to 90 degrees
- moved R61 193.3 mm to (114.3, 34.5), turned to 270 degrees
- moved R62 191.8 mm to (113.8, 22.4), turned to 90 degrees
- moved C52 188.8 mm to (103.5, 28.7), turned to 180 degrees
- moved R76 188.7 mm to (111.8, 22.4), turned to 90 degrees
- moved R69 188.4 mm to (116.8, 23.4), turned to 180 degrees
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
Commit message: place LFO footprints
Parts:
- removed R100, R101, R102, R95, R96, R97, R98, R99: R, digikey-footprints:0805
- moved R80 340.2 mm to (70.6, 138.2), turned to 270 degrees
- moved R82 332.5 mm to (66.0, 134.6), turned to 180 degrees
- moved R86 328.9 mm to (74.7, 135.6), turned to 270 degrees
- moved R84 327.8 mm to (71.6, 144.3), turned to 180 degrees
- moved R85 317.2 mm to (71.6, 146.3), turned to 180 degrees
- moved R81 311.8 mm to (70.6, 134.6)
- moved C71 306.5 mm to (83.3, 144.8)
- moved R87 293.5 mm to (83.8, 122.9)
- moved C72 293.0 mm to (79.8, 136.1)
- moved C70 287.7 mm to (65.0, 141.2), turned to 270 degrees
- moved C73 269.2 mm to (83.8, 128.5)
- moved D2 263.3 mm to (75.7, 145.3)
- moved C17 25.5 mm to (74.7, 116.3)
- moved R17 25.5 mm to (72.1, 123.4)
- moved R18 25.5 mm to (76.7, 123.4)
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
Commit message: place filter footprints
Parts:
- moved R13 229.3 mm to (143.3, 111.8)
- moved R16 228.9 mm to (143.3, 98.0)
- moved C8 224.6 mm to (151.4, 98.0), turned to 90 degrees
- moved R10 223.4 mm to (156.5, 111.8), turned to 90 degrees
- moved R7 222.4 mm to (160.0, 94.0)
- moved C12 221.4 mm to (149.4, 98.0), turned to 90 degrees
- moved C9 220.8 mm to (149.4, 111.8), turned to 270 degrees
- moved R5 220.3 mm to (150.4, 115.3), turned to 180 degrees
- moved R12 219.7 mm to (153.4, 98.0), turned to 270 degrees
- moved R9 219.5 mm to (153.4, 111.8), turned to 90 degrees
- moved R2 218.5 mm to (151.9, 143.3), turned to 180 degrees
- moved R8 216.8 mm to (148.8, 94.0), turned to 180 degrees
- moved C16 216.6 mm to (144.3, 102.1), turned to 180 degrees
- moved R4 215.4 mm to (159.0, 143.3)
- moved C7 213.6 mm to (158.5, 98.0), turned to 90 degrees
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
Commit message: place envelope footprints. all footprints loosely grouped together.
Parts:
- moved R83 369.9 mm to (27.4, 87.4), turned to 180 degrees
- moved C68 204.3 mm to (109.2, 21.3)
- moved C30 197.5 mm to (428.8, 186.9)
- moved C31 191.7 mm to (428.8, 178.3)
- moved R78 186.7 mm to (109.2, 23.4)
- moved C26 173.6 mm to (420.6, 126.0)
- moved R29 169.7 mm to (420.1, 185.4)
- moved Q2 164.3 mm to (415.5, 188.4), turned to 270 degrees
- moved C27 162.0 mm to (420.6, 134.6)
- moved R21 154.3 mm to (408.9, 127.5), turned to 180 degrees
- moved C21 137.7 mm to (411.0, 182.6), turned to 90 degrees
- moved RV6 133.3 mm to (411.0, 189.0)
- moved Q3 129.6 mm to (408.9, 124.5), turned to 90 degrees
- moved RV7 129.6 mm to (404.4, 122.9), turned to 180 degrees
- moved R26 126.8 mm to (420.1, 187.5)
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Connections:
- R88 pad 1: Net-(R88-Pad1) -> /LFO Modulation and Routing/main_lfo

Commit message: add LFO mod pots to control board and fix pot placement
Parts:
- moved C28 27.7 mm to (351.5, 148.8)
- moved C29 27.7 mm to (351.5, 140.2)
- moved R24 27.7 mm to (343.9, 148.8)
- moved R34 27.7 mm to (343.9, 144.8)
- moved R33 27.7 mm to (343.9, 146.8)
- moved C23 27.7 mm to (334.8, 149.1)
- moved R22 27.7 mm to (339.3, 150.4)
- moved Q4 27.7 mm to (339.3, 147.3)
- moved R42 27.7 mm to (343.9, 142.7)
- moved RV8 27.7 mm to (339.3, 142.7)
- moved C20 24.9 mm to (355.1, 171.7)
- moved C24 24.9 mm to (338.0, 173.5)
- moved C25 24.9 mm to (338.0, 182.2)
- moved Q1 24.9 mm to (350.5, 177.3)
- moved R19 24.9 mm to (350.5, 174.2)
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
Commit message: route traces to bypass caps on MCU. control board and connectors are WIP.
Parts:
- removed RV18, RV19, RV20, RV21: 10kA, Potentiometers:Potentiometer_Bourns_PTV09A-1_Horizontal
- added J12: Conn_01x08, Pin_Headers:Pin_Header_Straight_1x08_Pitch2.54mm, F.Cu at (224.3, 33.8)
- moved C77 190.3 mm to (254.8, 31.8)
- moved R89 190.3 mm to (248.2, 33.8)
- moved R90 190.3 mm to (248.2, 46.5)
- moved U5 190.3 mm to (246.9, 40.2)
- moved C74 190.3 mm to (239.0, 31.8)
- moved C75 190.3 mm to (239.0, 49.0)
- moved C76 190.3 mm to (254.8, 49.0)
- moved R88 190.3 mm to (245.6, 46.4)
- moved R91 190.3 mm to (245.6, 33.8)
- moved R23 97.5 mm to (324.6, 109.7)
- moved C23 97.5 mm to (242.3, 118.1)
- moved C24 97.5 mm to (245.6, 142.5)
- moved C25 97.5 mm to (245.6, 151.2)
- moved C28 97.5 mm to (259.1, 117.9)
- moved C29 97.5 mm to (259.1, 109.2)
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Connections:
- C74 pad 2: Net-(C74-Pad2) -> /LFO Modulation and Routing/lfo_in_3
- C75 pad 2: Net-(C75-Pad2) -> /LFO Modulation and Routing/lfo_in_1
- C76 pad 2: Net-(C76-Pad2) -> /LFO Modulation and Routing/lfo_in_2
- C77 pad 2: Net-(C77-Pad2) -> /LFO Modulation and Routing/lfo_in_4
Routing:
- net GNDD: track 0.00 -> 96.5 mm, vias 0 -> 3
- net +5V: track 0.00 -> 83.7 mm, vias 0 -> 4
- net Net-(C82-Pad1): track 0.00 -> 22.6 mm
- net Net-(C87-Pad1): track 0.00 -> 22.4 mm
- net /Microcontroller/XRES: track 0.00 -> 12.3 mm
- net Net-(J7-Pad4): track 0.00 -> 9.84 mm
- net /Connectors/envelope_pwm_bypass_in_4: track 0.00 -> 9.45 mm
- net /Connectors/envelope_pwm_bypass_in_1: track 0.00 -> 9.09 mm
- net Net-(C88-Pad1): track 0.00 -> 8.94 mm
- net /Connectors/envelope_pwm_bypass_in_3: track 0.00 -> 8.55 mm
- net /Connectors/envelope_pwm_bypass_in_2: track 0.00 -> 8.44 mm
- net Net-(J7-Pad3): track 0.00 -> 7.88 mm
- net /Microcontroller/envelope_pwm_1: track 0.00 -> 7.26 mm
- net /Microcontroller/envelope_pwm_4: track 0.00 -> 6.89 mm
- net Net-(J7-Pad2): track 0.00 -> 5.93 mm
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Other:
- rule trace_min: 0.2 -> 0.0889
- rule via_min_drill: 0.3 -> 0.2
- rule via_min_size: 0.4 -> 0.45

Commit message: route connectors on control board. Will add additional set of connectors for filter knobs to simplify routing.
Parts:
- removed J10, J11, J8, J9: Conn_01x13, Pin_Headers:Pin_Header_Straight_1x13_Pitch2.54mm
- moved C26 264.3 mm to (90.4, 3.56), turned to 90 degrees
- moved C27 260.1 mm to (99.1, 3.56), turned to 90 degrees
- moved R23 254.5 mm to (89.9, 11.2), turned to 90 degrees
- moved R31 253.5 mm to (91.9, 11.2), turned to 90 degrees
- moved R32 252.4 mm to (94.0, 11.2), turned to 90 degrees
- moved R41 251.4 mm to (96.0, 11.2), turned to 270 degrees
- moved Q3 249.8 mm to (88.9, 15.2), turned to 180 degrees
- moved R21 248.1 mm to (91.9, 15.2), turned to 270 degrees
- moved RV7 244.7 mm to (87.4, 19.8), turned to 270 degrees
- moved C22 240.4 mm to (94.0, 20.3), turned to 0 degrees
- moved C30 222.0 mm to (123.8, 87.9), turned to 270 degrees
- moved C34 221.7 mm to (99.1, 32.5), turned to 90 degrees
- moved R45 220.6 mm to (101.1, 32.5), turned to 270 degrees
- moved Q7 219.5 mm to (107.7, 31.0), turned to 180 degrees
- moved R37 218.1 mm to (110.7, 31.0), turned to 90 degrees
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Connections:
- U1 pad 1: Net-(C13-Pad1) -> Net-(C10-Pad1)
- U1 pad 10: Net-(C7-Pad1) -> Net-(C8-Pad1)
- U1 pad 12: Net-(C8-Pad1) -> Net-(C7-Pad1)
- U1 pad 13: Net-(C12-Pad1) -> Net-(C11-Pad1)
- U1 pad 14: Net-(C12-Pad1) -> Net-(C11-Pad1)
- U1 pad 2: Net-(C13-Pad1) -> Net-(C10-Pad1)
- U1 pad 3: Net-(C5-Pad1) -> Net-(C6-Pad1)
- U1 pad 5: Net-(C6-Pad1) -> Net-(C5-Pad1)
- U1 pad 6: Net-(C10-Pad1) -> Net-(C13-Pad1)
- U1 pad 7: Net-(C10-Pad1) -> Net-(C13-Pad1)
- U1 pad 8: Net-(C11-Pad1) -> Net-(C12-Pad1)
- U1 pad 9: Net-(C11-Pad1) -> Net-(C12-Pad1)
- U2 pad 1: Net-(C40-Pad1) -> Net-(C41-Pad1)
- U2 pad 2: Net-(C40-Pad1) -> Net-(C41-Pad1)
- U2 pad 3: Net-(C36-Pad1) -> Net-(C37-Pad1)
- U2 pad 5: Net-(C37-Pad1) -> Net-(C36-Pad1)
- U2 pad 6: Net-(C41-Pad1) -> Net-(C40-Pad1)
- U2 pad 7: Net-(C41-Pad1) -> Net-(C40-Pad1)
Routing:
- net /Filters/osc4: track 0.00 -> 40.7 mm
- net /Filters/osc3: track 0.00 -> 23.1 mm, vias 0 -> 2
- net /Filters/osc2: track 0.00 -> 13.9 mm
- net /Microcontroller/SDAT: track 0.00 -> 13.1 mm, vias 0 -> 1
- net /Microcontroller/SCLK: track 0.00 -> 12.6 mm, vias 0 -> 1
- net Net-(C13-Pad1): track 0.00 -> 12.3 mm
- net Net-(C6-Pad1): track 0.00 -> 10.3 mm
- net Net-(C5-Pad1): track 0.00 -> 8.99 mm
- net Net-(C36-Pad1): track 0.00 -> 8.39 mm
- net /Filters/osc1: track 0.00 -> 8.39 mm
- net Net-(C37-Pad1): track 0.00 -> 8.34 mm
- net Net-(C30-Pad1): track 0.00 -> 7.41 mm
- net Net-(C21-Pad1): track 0.00 -> 6.83 mm
- net Net-(C31-Pad1): track 0.00 -> 5.62 mm
- net /Envelope/lfo_bias_2: track 0.00 -> 4.53 mm
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