File: Hardware/Synth Engine/synth_psoc.sch (KiCad schematic (older format))
At the start: 0 parts

Commit message: fix remaining connector placement. Routing still WIP
Changed lines of the file:
@@
 $EndSheet
 $Sheet
-S 8850 2450 600  800
+S 9150 2450 600  800
 U 5C357081
 F0 "Mixer and Effects" 60
 F1 "mixer.sch" 60
-F2 "osc1" I L 8850 2500 60
-F3 "osc2" I L 8850 2600 60
-F4 "osc3" I L 8850 2700 60
-F5 "osc4" I L 8850 2800 60
-$EndSheet
-$Sheet
-S 5300 4200 600  1500
-U 5C35738C
-F0 "LFO Modulation and Routing" 60
-F1 "lfo.sch" 60
-F2 "lfo1" O R 5900 4300 60
-F3 "lfo2" O R 5900 4400 60
-F4 "lfo3" O R 5900 4500 60
-F5 "lfo4" O R 5900 4600 60
-F6 "lfo_in_1" O R 5900 4800 60
-F7 "lfo_out_1" I R 5900 4900 60
-F8 "lfo_in_2" O R 5900 5000 60
-F9 "lfo_out_2" I R 5900 5100 60
-F10 "lfo_in_3" O R 5900 5200 60
-F11 "lfo_out_3" I R 5900 5300 60
-F12 "lfo_in_4" O R 5900 5400 60
-F13 "lfo_out_4" I R 5900 5500 60
+F2 "osc1" I L 9150 2500 60
+F3 "osc2" I L 9150 2600 60
+F4 "osc3" I L 9150 2700 60
+F5 "osc4" I L 9150 2800 60
+F6 "lfo_freq_in" O L 9150 3050 60
+F7 "lfo_freq_out" I L 9150 3150 60
 $EndSheet
 $Sheet
@@
 	5900 4300 7000 4300
 Wire Wire Line
-	8350 2800 8850 2800
-Wire Wire Line
-	8350 2700 8850 2700
-Wire Wire Line
-	8350 2600 8850 2600
-Wire Wire Line
-	8350 2500 8850 2500
+	8350 2800 9150 2800
+Wire Wire Line
+	8350 2700 9150 2700
+Wire Wire Line
+	8350 2600 9150 2600
+Wire Wire Line
+	8350 2500 9150 2500
 Wire Wire Line
 	6800 2800 7450 2800
@@
 Wire Wire Line
 	900  3250 950  3250
+$Sheet
+S 5250 4200 650  1600
+U 5C35738C
+F0 "LFO Modulation and Routing" 60
+F1 "lfo.sch" 60
+F2 "lfo1" O R 5900 4300 60
+F3 "lfo2" O R 5900 4400 60
+F4 "lfo3" O R 5900 4500 60
+F5 "lfo4" O R 5900 4600 60
+F6 "lfo_in_1" O R 5900 4800 60
+F7 "lfo_out_1" I R 5900 4900 60
+F8 "lfo_in_2" O R 5900 5000 60
+F9 "lfo_out_2" I R 5900 5100 60
+F10 "lfo_in_3" O R 5900 5200 60
+F11 "lfo_out_3" I R 5900 5300 60
+F12 "lfo_in_4" O R 5900 5400 60
+F13 "lfo_out_4" I R 5900 5500 60
+F14 "lfo_freq_in" O R 5900 5600 60
+F15 "lfo_freq_out" I R 5900 5700 60
+$EndSheet
+Text Label 6150 5700 0    60   ~ 0
+lfo_freq_out
+Text Label 6150 5600 0    60   ~ 0
+lfo_freq_in
+Wire Wire Line
+	6150 5700 5900 5700
+Wire Wire Line
+	5900 5600 6150 5600
+Text Label 9050 3050 2    60   ~ 0
+lfo_freq_in
+Text Label 9050 3150 2    60   ~ 0
+lfo_freq_out
+Wire Wire Line
+	9050 3050 9150 3050
+Wire Wire Line
+	9050 3150 9150 3150
 $EndSCHEMATC

Commit message: redo connector routing with 2-row connectors
Changed lines of the file:
@@
 F6 "lfo_freq_in" O L 9150 3050 60
 F7 "lfo_freq_out" I L 9150 3150 60
+F8 "mcu_delay_in" O R 9750 2850 60
+F9 "mcu_delay_out" I R 9750 2950 60
 $EndSheet
 $Sheet
@@
 F36 "envelope_pwm_bypass_out_3" I L 3650 6450 60
 F37 "envelope_pwm_bypass_out_4" I L 3650 7250 60
+F38 "mcu_delay_in" O L 3650 3900 60
+F39 "mcu_delay_out" I L 3650 4000 60
 $EndSheet
 $Sheet
@@
 Wire Wire Line
 	9050 3150 9150 3150
+Text Label 9900 2850 0    60   ~ 0
+mcu_delay_in
+Text Label 9900 2950 0    60   ~ 0
+mcu_delay_out
+Wire Wire Line
+	9900 2850 9750 2850
+Wire Wire Line
+	9750 2950 9900 2950
+Text Label 3500 3900 2    60   ~ 0
+mcu_delay_in
+Text Label 3500 4000 2    60   ~ 0
+mcu_delay_out
+Wire Wire Line
+	3500 3900 3650 3900
+Wire Wire Line
+	3500 4000 3650 4000
 $EndSCHEMATC

Commit message: redo second connector on main board
Changed lines of the file:
@@
 F38 "mcu_delay_in" O L 3650 3900 60
 F39 "mcu_delay_out" I L 3650 4000 60
+F40 "osc1_hold" I L 3650 4350 60
+F41 "osc2_hold" I L 3650 5150 60
+F42 "osc3_hold" I L 3650 5950 60
+F43 "osc4_hold" I L 3650 6750 60
 $EndSheet
 $Sheet
@@
 F48 "lfo_in_4" O L 950 3150 60
 F49 "lfo_out_4" I L 950 3250 60
+F50 "osc1_hold" O R 2800 4350 60
+F51 "osc2_hold" O R 2800 5150 60
+F52 "osc3_hold" O R 2800 5950 60
+F53 "osc4_hold" O R 2800 6750 60
 $EndSheet
 Wire Wire Line
@@
 Wire Wire Line
 	3500 4000 3650 4000
+Wire Wire Line
+	2800 4350 3650 4350
+Wire Wire Line
+	2800 5150 3650 5150
+Wire Wire Line
+	2800 5950 3650 5950
+Wire Wire Line
+	2800 6750 3650 6750
 $EndSCHEMATC
