File: Hardware/Synth Control Board/control_board.sch (KiCad schematic (older format))
At the start: 90 parts, among them J1 Conn_02x13_Odd_Even, J10 Conn_01x05, J11 Conn_01x08, J2 Conn_01x03, J3 Conn_02x13_Odd_Even, J4 Conn_01x08, J7 Conn_01x05, J8 Conn_01x05, J9 Conn_01x05, SW1 SW_DPDT_x2, SW10 SW_SPST, SW11 SW_SPST, SW12 SW_SPST, SW13 SW_SPST, SW2 SW_SPST, SW3 SW_SPST, SW4 SW_SPST, SW5 SW_SPST, SW6 SW_SPDT, SW7 SW_SPDT, SW8 SW_SPDT, SW9 SW_SPDT

Commit message: fix some missing traces on main board
Parts:
- SW6, SW7, SW8, SW9: footprint SparkFun-Electromechanical:SWITCH-SPDT -> switches:switch_toggle_4.7mm_pitch
Changed lines of the file:
@@
 F 0 "SW9" H 8700 770 50  0000 C CNN
 F 1 "SW_SPDT" H 8700 400 50  0000 C CNN
-F 2 "SparkFun-Electromechanical:SWITCH-SPDT" H 8700 600 50  0001 C CNN
+F 2 "switches:switch_toggle_4.7mm_pitch" H 8700 600 50  0001 C CNN
 F 3 "" H 8700 600 50  0001 C CNN
 	1    8700 600
@@
 F 0 "SW8" H 8700 1170 50  0000 C CNN
 F 1 "SW_SPDT" H 8700 800 50  0000 C CNN
-F 2 "SparkFun-Electromechanical:SWITCH-SPDT" H 8700 1000 50  0001 C CNN
+F 2 "switches:switch_toggle_4.7mm_pitch" H 8700 1000 50  0001 C CNN
 F 3 "" H 8700 1000 50  0001 C CNN
 	1    8700 1000
@@
 F 0 "SW7" H 8700 1470 50  0000 C CNN
 F 1 "SW_SPDT" H 8700 1100 50  0000 C CNN
-F 2 "SparkFun-Electromechanical:SWITCH-SPDT" H 8700 1300 50  0001 C CNN
+F 2 "switches:switch_toggle_4.7mm_pitch" H 8700 1300 50  0001 C CNN
 F 3 "" H 8700 1300 50  0001 C CNN
 	1    8700 1300
@@
 F 0 "SW6" H 8700 1770 50  0000 C CNN
 F 1 "SW_SPDT" H 8700 1400 50  0000 C CNN
-F 2 "SparkFun-Electromechanical:SWITCH-SPDT" H 8700 1600 50  0001 C CNN
+F 2 "switches:switch_toggle_4.7mm_pitch" H 8700 1600 50  0001 C CNN
 F 3 "" H 8700 1600 50  0001 C CNN
 	1    8700 1600
@@
 Connection ~ 4250 5950
 Wire Wire Line
-	4100 5950 4250 5950
-Wire Wire Line
-	4250 5950 4300 5950
+	4100 5950 4300 5950
 Wire Wire Line
 	4250 6150 4250 5950
@@
 	2600 6300 2700 6300
 Wire Wire Line
-	1800 6300 1800 6300
-Wire Wire Line
-	1800 6300 1950 6300
-Wire Wire Line
-	1950 6300 2000 6300
+	1800 6300 2000 6300
 Wire Wire Line
 	1950 6050 2300 6050
 Connection ~ 1150 6300
 Wire Wire Line
-	1000 6300 1150 6300
-Wire Wire Line
-	1150 6300 1200 6300
+	1000 6300 1200 6300
 Wire Wire Line
 	1150 6050 1150 6300
@@
 	2300 6050 2300 6100
 Wire Wire Line
-	950  6850 1050 6850
-Wire Wire Line
-	1050 6850 1100 6850
-Wire Wire Line
-	1700 6850 1800 6850
-Wire Wire Line
-	1800 6850 1900 6850
-Wire Wire Line
-	1900 6850 1950 6850
+	950  6850 1100 6850
+Wire Wire Line
+	1700 6850 1950 6850
 Wire Wire Line
 	1400 6650 1400 6600
@@
 Connection ~ 1900 6850
 Wire Wire Line
-	950  7350 1050 7350
-Wire Wire Line
-	1050 7350 1100 7350
+	950  7350 1100 7350
 Wire Wire Line
 	1400 7150 1400 7100
@@
 Connection ~ 1050 7350
 Wire Wire Line
-	1700 7350 1800 7350
-Wire Wire Line
-	1800 7350 1900 7350
-Wire Wire Line
-	1900 7350 1950 7350
+	1700 7350 1950 7350
 Wire Wire Line
 	1800 7050 1800 7350
@@
 	2550 7350 2750 7350
 Wire Wire Line
-	950  7800 1050 7800
-Wire Wire Line
-	1050 7800 1100 7800
+	950  7800 1100 7800
 Wire Wire Line
 	1400 7600 1400 7550
@@
 Connection ~ 1050 7800
 Wire Wire Line
-	1700 7800 1800 7800
-Wire Wire Line
-	1800 7800 1900 7800
-Wire Wire Line
-	1900 7800 1950 7800
+	1700 7800 1950 7800
 Wire Wire Line
 	1800 7500 1800 7800

Commit message: add MIDI
Parts:
- SW1, SW10, SW11, SW12, SW13, SW2, SW3, SW4, SW5: footprint SparkFun-Electromechanical:SWITCH-SPDT -> switches:switch_toggle_4.7mm_pitch
Changed lines of the file:
@@
 F 0 "SW3" H 6400 1225 50  0000 C CNN
 F 1 "SW_SPST" H 6400 1000 50  0000 C CNN
-F 2 "SparkFun-Electromechanical:SWITCH-SPDT" H 6400 1100 50  0001 C CNN
+F 2 "switches:switch_toggle_4.7mm_pitch" H 6400 1100 50  0001 C CNN
 F 3 "" H 6400 1100 50  0001 C CNN
 	1    6400 1100
@@
 F 0 "SW4" H 6400 1325 50  0000 C CNN
 F 1 "SW_SPST" H 6400 1100 50  0000 C CNN
-F 2 "SparkFun-Electromechanical:SWITCH-SPDT" H 6400 1200 50  0001 C CNN
+F 2 "switches:switch_toggle_4.7mm_pitch" H 6400 1200 50  0001 C CNN
 F 3 "" H 6400 1200 50  0001 C CNN
 	1    6400 1200
@@
 F 0 "SW2" H 6400 1125 50  0000 C CNN
 F 1 "SW_SPST" H 6400 900 50  0000 C CNN
-F 2 "SparkFun-Electromechanical:SWITCH-SPDT" H 6400 1000 50  0001 C CNN
+F 2 "switches:switch_toggle_4.7mm_pitch" H 6400 1000 50  0001 C CNN
 F 3 "" H 6400 1000 50  0001 C CNN
 	1    6400 1000
@@
 F 0 "SW5" H 6400 1425 50  0000 C CNN
 F 1 "SW_SPST" H 6400 1200 50  0000 C CNN
-F 2 "SparkFun-Electromechanical:SWITCH-SPDT" H 6400 1300 50  0001 C CNN
+F 2 "switches:switch_toggle_4.7mm_pitch" H 6400 1300 50  0001 C CNN
 F 3 "" H 6400 1300 50  0001 C CNN
 	1    6400 1300
@@
 F 0 "SW1" H 3750 6820 50  0000 C CNN
 F 1 "SW_DPDT_x2" H 4000 6650 50  0000 C CNN
-F 2 "SparkFun-Electromechanical:SWITCH-SPDT" H 3750 6650 50  0001 C CNN
+F 2 "switches:switch_toggle_4.7mm_pitch" H 3750 6650 50  0001 C CNN
 F 3 "" H 3750 6650 50  0001 C CNN
 	1    3750 6650
@@
 F 0 "SW11" H 10550 1175 50  0000 C CNN
 F 1 "SW_SPST" H 10550 950 50  0000 C CNN
-F 2 "SparkFun-Electromechanical:SWITCH-SPDT" H 10550 1050 50  0001 C CNN
+F 2 "switches:switch_toggle_4.7mm_pitch" H 10550 1050 50  0001 C CNN
 F 3 "" H 10550 1050 50  0001 C CNN
 	1    10550 1050
@@
 F 0 "SW12" H 10550 1275 50  0000 C CNN
 F 1 "SW_SPST" H 10550 1050 50  0000 C CNN
-F 2 "SparkFun-Electromechanical:SWITCH-SPDT" H 10550 1150 50  0001 C CNN
+F 2 "switches:switch_toggle_4.7mm_pitch" H 10550 1150 50  0001 C CNN
 F 3 "" H 10550 1150 50  0001 C CNN
 	1    10550 1150
@@
 F 0 "SW10" H 10550 1075 50  0000 C CNN
 F 1 "SW_SPST" H 10550 850 50  0000 C CNN
-F 2 "SparkFun-Electromechanical:SWITCH-SPDT" H 10550 950 50  0001 C CNN
+F 2 "switches:switch_toggle_4.7mm_pitch" H 10550 950 50  0001 C CNN
 F 3 "" H 10550 950 50  0001 C CNN
 	1    10550 950
@@
 F 0 "SW13" H 10550 1375 50  0000 C CNN
 F 1 "SW_SPST" H 10550 1150 50  0000 C CNN
-F 2 "SparkFun-Electromechanical:SWITCH-SPDT" H 10550 1250 50  0001 C CNN
+F 2 "switches:switch_toggle_4.7mm_pitch" H 10550 1250 50  0001 C CNN
 F 3 "" H 10550 1250 50  0001 C CNN
 	1    10550 1250
