File: Hardware/Synth_Engine/vca.sch (KiCad schematic (older format))
At the start: 70 parts, among them J4 Conn_01x08, Q1 MMBT3904-TP, Q2 MMBT3904-TP, Q3 MMBT3904-TP, Q4 MMBT3904-TP, Q5 MMBFJ177, Q6 MMBFJ177, Q7 MMBFJ177, Q8 MMBFJ177, U2 TL074

Commit message: update BOM for v2 sample.
Parts:
- C24, C25, C26, C27, C28, C29, C30, C31: value 220u -> 220uF
Changed lines of the file:
@@
 P 5600 1700
 F 0 "C24" H 5610 1770 50  0000 L CNN
-F 1 "220u" H 5610 1620 50  0000 L CNN
+F 1 "220uF" H 5610 1620 50  0000 L CNN
 F 2 "Capacitors_SMD:CP_Elec_8x10" H 5600 1700 50  0001 C CNN
 F 3 "" H 5600 1700 50  0001 C CNN
@@
 P 5700 3100
 F 0 "C30" H 5710 3170 50  0000 L CNN
-F 1 "220u" H 5710 3020 50  0000 L CNN
+F 1 "220uF" H 5710 3020 50  0000 L CNN
 F 2 "Capacitors_SMD:CP_Elec_8x10" H 5700 3100 50  0001 C CNN
 F 3 "" H 5700 3100 50  0001 C CNN
@@
 P 5600 4350
 F 0 "C26" H 5610 4420 50  0000 L CNN
-F 1 "220u" H 5610 4270 50  0000 L CNN
+F 1 "220uF" H 5610 4270 50  0000 L CNN
 F 2 "Capacitors_SMD:CP_Elec_8x10" H 5600 4350 50  0001 C CNN
 F 3 "" H 5600 4350 50  0001 C CNN
@@
 P 5600 5700
 F 0 "C28" H 5610 5770 50  0000 L CNN
-F 1 "220u" H 5610 5620 50  0000 L CNN
+F 1 "220uF" H 5610 5620 50  0000 L CNN
 F 2 "Capacitors_SMD:CP_Elec_8x10" H 5600 5700 50  0001 C CNN
 F 3 "" H 5600 5700 50  0001 C CNN
@@
 P 5600 5900
 F 0 "C29" H 5610 5970 50  0000 L CNN
-F 1 "220u" H 5610 5820 50  0000 L CNN
+F 1 "220uF" H 5610 5820 50  0000 L CNN
 F 2 "Capacitors_SMD:CP_Elec_8x10" H 5600 5900 50  0001 C CNN
 F 3 "" H 5600 5900 50  0001 C CNN
@@
 P 5600 1900
 F 0 "C25" H 5610 1970 50  0000 L CNN
-F 1 "220u" H 5610 1820 50  0000 L CNN
+F 1 "220uF" H 5610 1820 50  0000 L CNN
 F 2 "Capacitors_SMD:CP_Elec_8x10" H 5600 1900 50  0001 C CNN
 F 3 "" H 5600 1900 50  0001 C CNN
@@
 P 5700 3300
 F 0 "C31" H 5710 3370 50  0000 L CNN
-F 1 "220u" H 5710 3220 50  0000 L CNN
+F 1 "220uF" H 5710 3220 50  0000 L CNN
 F 2 "Capacitors_SMD:CP_Elec_8x10" H 5700 3300 50  0001 C CNN
 F 3 "" H 5700 3300 50  0001 C CNN
@@
 P 5600 4550
 F 0 "C27" H 5610 4620 50  0000 L CNN
-F 1 "220u" H 5610 4470 50  0000 L CNN
+F 1 "220uF" H 5610 4470 50  0000 L CNN
 F 2 "Capacitors_SMD:CP_Elec_8x10" H 5600 4550 50  0001 C CNN
 F 3 "" H 5600 4550 50  0001 C CNN
