File: Hardware/Synth_Engine/mixer.sch (KiCad schematic (older format))
At the start: 61 parts, among them J2 Audio-Jack-2_Switch, J5 Conn_01x08, U3 TL074, U8 PT2399

Commit message: update BOM for v2 sample.
Parts:
- C64: value 0.01uF -> 10nF
Changed lines of the file:
@@
 P 6850 2400
 F 0 "C64" H 6860 2470 50  0000 L CNN
-F 1 "0.01uF" H 6860 2320 50  0000 L CNN
+F 1 "10nF" H 6860 2320 50  0000 L CNN
 F 2 "digikey-footprints:0805" H 6850 2400 50  0001 C CNN
 F 3 "" H 6850 2400 50  0001 C CNN

Commit message: reduce delay FB end stop resistor.
Parts:
- R73: value 10k -> 4.7k
Changed lines of the file:
@@
 P 7700 2450
 F 0 "R73" V 7780 2450 50  0000 C CNN
-F 1 "10k" V 7700 2450 50  0000 C CNN
+F 1 "4.7k" V 7700 2450 50  0000 C CNN
 F 2 "digikey-footprints:0805" V 7630 2450 50  0001 C CNN
 F 3 "" H 7700 2450 50  0001 C CNN
